Commit message: feat: introduce pallet truck with aruco label

File: simulation/infobot_agent/urdf/infobot.urdf.xacro (robot description, xacro)
@@ -8,3 +8,4 @@
     <xacro:include filename="sensors.xacro" />
     <xacro:include filename="infobot.gazebo.xacro"/>
+    <xacro:include filename="aruco.xacro"/>
 </robot>

File: simulation/infobot_agent/urdf/links.xacro (robot description, xacro)
@@ -4,31 +4,31 @@
     <link name="base_link">
         <visual>
-            <xacro:if value="${robot_type == 'GOPAL400'}">
-                <origin xyz="0 0 0" rpy="0 0 0" />
-                <geometry>
-                    <mesh filename="file://$(find infobot_agent)/models/infobot_common/meshes/AMR_GP400.dae" scale="1 1 1"/>
-                    <!-- <box size="${base_length} ${base_width} ${base_height}" /> -->
-                </geometry>
-            </xacro:if>
-            <xacro:if value="${robot_type == 'FORKLIFT'}">
-                <origin xyz="-1.5 -0.535 0" rpy="0 0 0" />
-                <geometry>
-                    <mesh filename="file://$(find simlan_gazebo_environment)/models/forklift_robot/forklift_robot_description/meshes/base_link.dae"/>
-                </geometry>
-            </xacro:if>
+<xacro:if value="${robot_type == 'GOPAL400'}">
+            <origin xyz="0 0 0" rpy="0 0 0" />
+            <geometry>
+                <mesh filename="file://$(find infobot_agent)/models/infobot_common/meshes/VOLVO_AVG.dae" scale="1 1 1"/>
+                <!-- <box size="${base_length} ${base_width} ${base_height}" /> -->
+            </geometry>
+</xacro:if>
+<xacro:if value="${robot_type == 'FORKLIFT'}">
+            <origin xyz="-1.5 -0.5 0" rpy="0 0 0" />
+            <geometry>
+                <mesh filename="file://$(find simlan_gazebo_environment)/models/forklift_robot/forklift_robot_description/meshes/base_link.dae"/>
+            </geometry>
+</xacro:if>
         </visual>
         <collision>
-            <xacro:if value="${robot_type == 'GOPAL400'}">
-                <geometry>
-                    <mesh filename="file://$(find infobot_agent)/models/infobot_common/meshes/AMR_GP400.dae" scale="1 1 1"/>
-                    <!-- <box size="${base_length} ${base_width} ${base_height}" />  -->
-                </geometry>
-            </xacro:if>
-            <xacro:if value="${robot_type == 'FORKLIFT'}">
-                <origin xyz="-1.5 -0.535 0" rpy="0 0 0" />
-                <geometry>
-                    <mesh filename="file://$(find simlan_gazebo_environment)/models/forklift_robot/forklift_robot_description/meshes/base_link.dae"/>
-                </geometry>
-            </xacro:if>
+<xacro:if value="${robot_type == 'GOPAL400'}">
+            <geometry>
+                <mesh filename="file://$(find infobot_agent)/models/infobot_common/meshes/VOLVO_AVG.dae" scale="1 1 1"/>
+                <!-- <box size="${base_length} ${base_width} ${base_height}" />  -->
+            </geometry>
+</xacro:if>
+<xacro:if value="${robot_type == 'FORKLIFT'}">
+            <origin xyz="-1.5 -0.5 0" rpy="0 0 0" />
+            <geometry>
+                <mesh filename="file://$(find simlan_gazebo_environment)/models/forklift_robot/forklift_robot_description/meshes/base_link.dae"/>
+            </geometry>
+</xacro:if>
         </collision>
         <xacro:inertial_box m="${base_mass}"  d="${base_length}" w="${base_width}" h="${base_height}"/>
@@ -45,5 +45,5 @@
             <collision>
                 <geometry>
-                    <sphere radius="${wheel_radius*wheel_radius_multiple}" />
+                    <cylinder length="${wheel_width}" radius="${wheel_radius*wheel_radius_multiple}" />
                 </geometry>
             </collision>

File: simulation/infobot_agent/urdf/properties.xacro (robot description, xacro)
@@ -1,5 +1,5 @@
 <?xml version="1.0"?>
 <robot xmlns:xacro="http://ros.org/wiki/xacro">
-<!-- GOPAL400 and FORKLIFT -->
+<!-- VOLVO_GPSS_ARHO and FORKLIFT -->
 <xacro:property name="robot_type" value="FORKLIFT"/>
     <xacro:property name="base_length" value="1.4"/>

File: simulation/static_agent_launcher/description/camera_config.xacro (robot description, xacro)
@@ -2,4 +2,4 @@
 <!-- =================================== -->
 <robot xmlns:xacro="http://www.ros.org/wiki/xacro">
-<xacro:camera number="164" x="19.018611699231805" y="0.5996158690202326" z="7.312413251033551" r="1.5198482458361036" p="1.2025224147143143" w="2.9981981711263943" width="256" height="256" k1="-0.3851544658419547" k2="0.2065606446662026" k3="-0.06703301309031716" p1="-8.882469357164693e-05" p2="-0.0002282099854856601" horizental_fov="1.4620172315943898" aspect_ratio="1"  />
+<xacro:camera number="164" x="19.018611699231805" y="0.5996158690202326" z="7.312413251033551" r="1.5198482458361036" p="1.2025224147143143" w="2.9981981711263943" width="3840" height="2160" k1="-0.3851544658419547" k2="0.2065606446662026" k3="-0.06703301309031716" p1="-8.882469357164693e-05" p2="-0.0002282099854856601" horizental_fov="1.4620172315943898" aspect_ratio="1.5623518885162968"  />
 </robot>
