Commit message: fix: sync gitlab with github

File: simulation/infobot_agent/urdf/infobot.gazebo.xacro (robot description, xacro)
@@ -101,5 +101,5 @@
           </scan>
           <range>
-            <min>0.120000</min>
+            <min>0.2</min>
             <max>50</max>
             <resolution>1</resolution>

File: simulation/infobot_agent/urdf/links.xacro (robot description, xacro)
@@ -4,31 +4,31 @@
     <link name="base_link">
         <visual>
-            <xacro:if value="${robot_type == 'GOPAL400'}">
-                <origin xyz="0 0 0" rpy="0 0 0" />
-                <geometry>
-                    <mesh filename="file://$(find infobot_agent)/models/infobot_common/meshes/AMR_GP400.dae" scale="1 1 1"/>
-                    <!-- <box size="${base_length} ${base_width} ${base_height}" /> -->
-                </geometry>
-            </xacro:if>
-            <xacro:if value="${robot_type == 'FORKLIFT'}">
-                <origin xyz="-1.5 -0.535 0" rpy="0 0 0" />
-                <geometry>
-                    <mesh filename="file://$(find simlan_gazebo_environment)/models/forklift_robot/forklift_robot_description/meshes/base_link.dae"/>
-                </geometry>
-            </xacro:if>
+<xacro:if value="${robot_type == 'GOPAL400'}">
+            <origin xyz="0 0 0" rpy="0 0 0" />
+            <geometry>
+                <mesh filename="file://$(find infobot_agent)/models/infobot_common/meshes/VOLVO_AVG.dae" scale="1 1 1"/>
+                <!-- <box size="${base_length} ${base_width} ${base_height}" /> -->
+            </geometry>
+</xacro:if>
+<xacro:if value="${robot_type == 'FORKLIFT'}">
+            <origin xyz="-1.5 -0.5 0" rpy="0 0 0" />
+            <geometry>
+                <mesh filename="file://$(find simlan_gazebo_environment)/models/forklift_robot/forklift_robot_description/meshes/base_link.dae"/>
+            </geometry>
+</xacro:if>
         </visual>
         <collision>
-            <xacro:if value="${robot_type == 'GOPAL400'}">
-                <geometry>
-                    <mesh filename="file://$(find infobot_agent)/models/infobot_common/meshes/AMR_GP400.dae" scale="1 1 1"/>
-                    <!-- <box size="${base_length} ${base_width} ${base_height}" />  -->
-                </geometry>
-            </xacro:if>
-            <xacro:if value="${robot_type == 'FORKLIFT'}">
-                <origin xyz="-1.5 -0.535 0" rpy="0 0 0" />
-                <geometry>
-                    <mesh filename="file://$(find simlan_gazebo_environment)/models/forklift_robot/forklift_robot_description/meshes/base_link.dae"/>
-                </geometry>
-            </xacro:if>
+<xacro:if value="${robot_type == 'GOPAL400'}">
+            <geometry>
+                <mesh filename="file://$(find infobot_agent)/models/infobot_common/meshes/VOLVO_AVG.dae" scale="1 1 1"/>
+                <!-- <box size="${base_length} ${base_width} ${base_height}" />  -->
+            </geometry>
+</xacro:if>
+<xacro:if value="${robot_type == 'FORKLIFT'}">
+            <origin xyz="-1.5 -0.5 0" rpy="0 0 0" />
+            <geometry>
+                <mesh filename="file://$(find simlan_gazebo_environment)/models/forklift_robot/forklift_robot_description/meshes/base_link.dae"/>
+            </geometry>
+</xacro:if>
         </collision>
         <xacro:inertial_box m="${base_mass}"  d="${base_length}" w="${base_width}" h="${base_height}"/>

File: simulation/infobot_agent/urdf/properties.xacro (robot description, xacro)
@@ -13,8 +13,8 @@
     <xacro:property name="scan_px" value="0.0"/>
     <xacro:property name="scan_py" value="0.0"/>
-    <xacro:property name="scan_pz" value="${base_height+0.5}"/>
+    <xacro:property name="scan_pz" value="${base_height+2.5}"/>
     <xacro:property name="camera_px" value="${base_length/2}"/>
     <xacro:property name="camera_py" value="0.0"/>
-    <xacro:property name="camera_pz" value="${base_height}"/>
+    <xacro:property name="camera_pz" value="${base_height+1.6}"/>
     <xacro:property name="infobot_friction" value="0.1"/>
     <xacro:property name="infobot_slip" value="0.0"/>
