Commit message: SIMLAN 2.0.0: Upgrade Gazebo from classic to ignition, Aruco_localization, GPSS Navigation, Bird's Eye View, Deprecating: Infobot

File: simulation/pallet_truck/pallet_truck_description/urdf/accessories/hokuyo_ust10.urdf.xacro (robot description, xacro)
@@ -15,9 +15,9 @@
       <gazebo reference="${frame}">
         <turnGravityOff>true</turnGravityOff>
-        <sensor type="ray" name="${frame}">
+        <sensor type="gpu_lidar" name="${frame}">
           <pose>0 0 0 0 0 0</pose>
           <visualize>false</visualize>
           <update_rate>${update_rate}</update_rate>
-          <ray>
+          <lidar>
             <scan>
               <horizontal>
@@ -38,13 +38,7 @@
               <stddev>0.001</stddev>
             </noise>
-          </ray>
-          <plugin name="gazebo_ros_laser" filename="libgazebo_ros_ray_sensor.so">
-            <ros>
-              <namespace>${robot_namespace}</namespace>
-              <remapping>~/out:=${topic}</remapping>
-            </ros>
-            <output_type>sensor_msgs/LaserScan</output_type>
-            <frame_name>${frame}</frame_name>
-          </plugin>
+          </lidar>
+          <topic>scan</topic>
+          <gz_frame_id>${frame}</gz_frame_id>
         </sensor>
       </gazebo>

File: simulation/pallet_truck/pallet_truck_description/urdf/aruco.xacro (robot description, xacro)
@@ -5,12 +5,12 @@
         <link name="aruco_${number}_link">
             <visual>
-                <origin xyz="0 0 0" rpy="0 0 0"/>
+                <origin xyz="0 0 0" rpy="0 0 ${PI}"/>
                 <geometry>
-                    <box size="0.5 0.5 .001"/>
+                    <box size="0.5 0.5 .001" comment="THE ACTUAL SIZE OF ARUCO"/>
                 </geometry>
             </visual>
         </link>
         <joint name="aruco_${number}_joint" type="fixed">
-            <origin xyz="-1.35 0 2.15" rpy="0 0 0"/>
+            <origin xyz="-0.8 0 1.30" rpy="0 0 0"/>
             <parent link="pallet_truck_base_link"/>
             <child link="aruco_${number}_link"/>
@@ -20,24 +20,16 @@
             <visual name="aruco_front_face">
                 <pose>0.00005 0 0 0 0 0</pose>
-                <geometry>
-                    <box>
-                        <size>0.0001 0.5 0.5</size>
-                    </box>
-                </geometry>
                 <material>
-                    <script>
-                        <uri>model://aruco/materials/scripts</uri>
-                        <uri>model://aruco/materials/textures</uri>
-                        <name>aruco_${number}</name>
-                    </script>
+                    <ambient>1 1 1 1</ambient>
+                    <diffuse>1 1 1 1</diffuse>
+                    <specular>0 0 0 0</specular>
+                    <emissive>0 0 0 0</emissive>
+                    <pbr>
+                        <metal>
+                            <albedo_map>model://aruco/materials/textures/12.png</albedo_map>
+                            <name>aruco_0</name>
+                        </metal>
+                    </pbr>
                 </material>
-            </visual>
-            <visual name="aruco_back_face">
-                <pose>-0.00005 0 0 0 0 0</pose>
-                <geometry>
-                    <box>
-                        <size>0.0001 0.5 0.5</size>
-                    </box>
-                </geometry>
             </visual>
         </gazebo>

File: simulation/pallet_truck/pallet_truck_description/urdf/pallet_truck.urdf.xacro (robot description, xacro)
@@ -21,4 +21,6 @@
   <material name="yellow"><color rgba="0.8 0.8 0.0 1.0" /></material>
   <material name="black"><color rgba="0.15 0.15 0.15 1.0" /></material>
+  <xacro:include filename="$(find pallet_truck_description)/urdf/aruco.xacro"/>
+  <xacro:include filename="$(find pallet_truck_description)/urdf/pallet_truck.gazebo" />
   <xacro:macro name="wheel" params="wheel_prefix *joint_pose">
     <link name="${wheel_prefix}_wheel_link">
@@ -84,4 +86,18 @@
     <origin xyz="${-wheelbase/2} ${-track/2} ${wheel_vertical_offset}" rpy="0 0 0" />
   </xacro:wheel>
+  <joint name="scan_joint" type="fixed">
+    <origin xyz="0 0 1.5" rpy="0 0 0"/>
+    <parent link="$(arg prefix)_base_link"/>
+    <child link="$(arg prefix)_scan_link"/>
+  </joint>
+  <!-- LIDAR -->
+  <link name="$(arg prefix)_scan_link">
+      <visual>
+      <origin xyz="0 0 0" rpy="0 0 0"/>
+      <geometry>
+          <box size="0.1 0.1 0.1"/>
+      </geometry>
+    </visual>
+  </link>
   <link name="$(arg prefix)_base_link"></link>
   <joint name="$(arg prefix)_base_link_joint" type="fixed">
@@ -94,12 +110,12 @@
       <origin xyz="0 0 0" rpy="0 0 0"/>
       <geometry>
-        <mesh filename="file://$(find pallet_truck_description)/meshes/VOLVO_AVG.dae" scale="1 1 1" />
-      </geometry>
-      <material name="dark_grey" />
+        <mesh filename="file://$(find pallet_truck_description)/meshes/VOLVO_AVG.dae" scale="0.6 0.6 0.6" />
+      </geometry>
+        <material name="black" />
     </visual>
     <collision>
       <origin xyz="0 0 0" rpy="0 0 0"/>
       <geometry>
-        <mesh filename="file://$(find pallet_truck_description)/meshes/VOLVO_AVG.dae" scale="1 1 1" />
+        <mesh filename="file://$(find pallet_truck_description)/meshes/VOLVO_AVG.dae" scale="0.6 0.6 0.6" />
       </geometry>
     </collision>
@@ -176,5 +192,5 @@
     <hardware>
       <xacro:if value="$(arg is_sim)">
-        <plugin>gazebo_ros2_control/GazeboSystem</plugin>
+        <plugin>gz_ros2_control/GazeboSimSystem</plugin>
       </xacro:if>
       <xacro:unless value="$(arg is_sim)">
@@ -206,5 +222,4 @@
   <!-- Bring in simulation data for Gazebo. -->
   <!-- <xacro:if value="$(arg is_sim)"> -->
-  <xacro:include filename="$(find pallet_truck_description)/urdf/pallet_truck.gazebo" />
   <!-- </xacro:if> -->
   <!-- Optional standard accessories, including their simulation data. The rendering
@@ -214,4 +229,3 @@
   <!-- Optional custom includes. -->
   <!--<xacro:include filename="$(optenv pallet_truck_URDF_EXTRAS empty.urdf)" />-->
-<xacro:include filename="$(find pallet_truck_description)/urdf/aruco.xacro"/>
 </robot>

File: simulation/static_agent_launcher/description/agents.urdf.xacro (robot description, xacro)
@@ -17,5 +17,5 @@
     </joint>
     <xacro:include filename="camera_config.xacro" />
-    <xacro:aruco number="1" x="9" y="9" z="0.001" r="0" p="0" w="0"/>
-    <xacro:aruco number="2" x="8" y="6" z="0.001" r="0" p="0" w="0"/>
+    <xacro:aruco number="1" x="7" y="3" z="0.001" r="0" p="0" w="0"/>
+    <xacro:aruco number="2" x="6" y="0" z="0.001" r="0" p="0" w="0"/>
 </robot>

File: simulation/static_agent_launcher/description/aruco_macros.xacro (robot description, xacro)
@@ -1,13 +1,13 @@
 <robot xmlns:xacro="http://www.ros.org/wiki/xacro">
     <xacro:macro name="aruco_link" params="number">
+        <static>true</static>
         <link name="aruco_${number}_link">
             <visual>
                 <origin xyz="0 0 0" rpy="0 0 0"/>
                 <geometry>
-                    <box size="0.5 0.5 .001"/>
+                    <box size="0.5 0.5 .001" comment="THE ACTUAL SIZE OF ARUCO"/>
                 </geometry>
             </visual>
         </link>
-        <xacro:inertial_box mass="0.1" x="0.12" y="0.15" z="0.15"/>
     </xacro:macro>
     <xacro:macro name="aruco_joint" params="attach_to number x y z r p w">
@@ -21,17 +21,17 @@
         <gazebo reference="aruco_${number}_link">
             <static>true</static>
-            <visual name="aruco_front_face">
+                <visual name="aruco_front_face">
                 <pose>0.00005 0 0 0 0 0</pose>
-                <geometry>
-                    <box>
-                        <size>0.0001 0.5 0.5</size>
-                    </box>
-                </geometry>
                 <material>
-                    <script>
-                        <uri>model://aruco/materials/scripts</uri>
-                        <uri>model://aruco/materials/textures</uri>
-                        <name>aruco_${number}</name>
-                    </script>
+                    <ambient>1 1 1 1</ambient>
+                    <diffuse>1 1 1 1</diffuse>
+                    <specular>0 0 0 0</specular>
+                    <emissive>0 0 0 0</emissive>
+                    <pbr>
+                        <metal>
+                            <albedo_map>model://aruco/materials/textures/${number}.png</albedo_map>
+                            <name>aruco_${number}</name>
+                        </metal>
+                    </pbr>
                 </material>
             </visual>
@@ -40,5 +40,5 @@
                 <geometry>
                     <box>
-                        <size>0.0001 0.5 0.5</size>
+                        <size>0.0001 1  1</size>
                     </box>
                 </geometry>

File: simulation/static_agent_launcher/description/camera_config.xacro (robot description, xacro)
@@ -2,4 +2,7 @@
 <!-- =================================== -->
 <robot xmlns:xacro="http://www.ros.org/wiki/xacro">
-<xacro:camera number="164" x="19.018611699231805" y="0.5996158690202326" z="7.312413251033551" r="1.5198482458361036" p="1.2025224147143143" w="2.9981981711263943" width="256" height="256" k1="-0.3851544658419547" k2="0.2065606446662026" k3="-0.06703301309031716" p1="-8.882469357164693e-05" p2="-0.0002282099854856601" horizental_fov="1.4620172315943898" aspect_ratio="1"  />
+<xacro:camera number="163" x="6.408863223463874" y="1.0584660310604614" z="7.292500745934433" r="1.26150086062305" p="1.5251520264293401" w="-0.3776042405847099" width="3840" height="2160" k1="-0.38583566587127305" k2="0.2099961443873393" k3="-0.07094931776988343" p1="9.279371221442497e-05" p2="0.00014849011979552266" horizontal_fov="1.4581859532350445" aspect_ratio="1.7777777777777777"  />
+<xacro:camera number="164" x="19.018611699231805" y="0.5996158690202326" z="7.312413251033551" r="1.5198482458361036" p="1.2025224147143143" w="2.9981981711263943" width="3840" height="2160" k1="-0.3851544658419547" k2="0.2065606446662026" k3="-0.06703301309031716" p1="-8.882469357164693e-05" p2="-0.0002282099854856601" horizontal_fov="1.4620172315943898" aspect_ratio="1.7777777777777777"  />
+<xacro:camera number="165" x="19.780977546074062" y="-3.598892158741938" z="7.320450325717852" r="0.21646481266366294" p="1.2312003431796872" w="0.13995159212967984" width="3840" height="2160" k1="-0.3856199901471728" k2="0.20812766168662827" k3="-0.0686518264523881" p1="-0.00023961544692403472" p2="-8.229104930400743e-05" horizontal_fov="1.4615731089914958" aspect_ratio="1.7777777777777777"  />
+<xacro:camera number="166" x="22.963270174027635" y="4.027979359238904" z="7.419277685692497" r="-1.0558178103115718" p="1.3797771301022628" w="-1.8322918256936183" width="3840" height="2160" k1="-0.38144336503488374" k2="0.19579882600150705" k3="-0.0586530291683016" p1="-0.0002683294214338217" p2="-2.68226954291596e-05" horizontal_fov="1.461834064552691" aspect_ratio="1.7777777777777777"  />
 </robot>

File: simulation/static_agent_launcher/description/camera_macros.xacro (robot description, xacro)
@@ -9,7 +9,7 @@
           </visual>
           <visual>
-              <origin xyz="0.03 0 0" rpy="0 ${pi/2} 0"/>
+              <origin xyz="0.00 0 0" rpy="0 ${pi/2} 0"/>
               <geometry>
-                  <cylinder length="0.06" radius="0.04" />
+                  <cylinder length="0.03" radius="0.04" />
               </geometry>
           </visual>
@@ -24,12 +24,15 @@
         </joint>
     </xacro:macro>
-    <xacro:macro name="camera_gazebo" params="number width height k1 k2 k3 p1 p2 horizental_fov aspect_ratio">
+    <xacro:macro name="camera_gazebo" params="number width height k1 k2 k3 p1 p2 horizontal_fov aspect_ratio">
         <gazebo reference="camera_${number}_link">
+            <!-- Camera Sensor -->
             <sensor name="camera_${number}" type="camera">
                 <always_on>true</always_on>
                 <visualize>true</visualize>
-                <update_rate>1</update_rate>
+                <update_rate>20</update_rate>
                 <camera name="intel_realsense_r200">
-                  <horizontal_fov>${horizental_fov}</horizontal_fov>
+                  <!-- <segmentation_type>instance</segmentation_type> -->
+                  <horizontal_fov>${horizontal_fov}</horizontal_fov>
+                  <camera_info_topic>camera_${number}/camera_info</camera_info_topic>
                   <aspect_ratio>${aspect_ratio}</aspect_ratio>
                   <image>
@@ -38,32 +41,92 @@
                     <format>R8G8B8</format>
                   </image>
-<!--
-                  <clip>
-                    <near>0.02</near>
-                    <far>300</far>
-                  </clip>
-                  <noise>
-                    <type>gaussian</type>
-                    <mean>0.0</mean>
-                    <stddev>0.007</stddev>
-                  </noise>
--->
-                    <distortion>
+                <lens>
+                    <radial_tangential>
                         <k1>${k1}</k1>
                         <k2>${k2}</k2>
-                        <k3>${k3}</k3>
                         <p1>${p1}</p1>
                         <p2>${p2}</p2>
-                    </distortion>
+                    </radial_tangential>
+                </lens>
                 </camera>
-                  <plugin name="camera_driver_${number}" filename="libgazebo_ros_camera.so">
-                  </plugin>
-              </sensor>
+                <topic>camera_${number}/image_raw</topic>
+                <gz_frame_id>camera_link_optical</gz_frame_id>
+            </sensor>
+            <!-- Depth camera sensor -->
+            <sensor name="depth_${number}" type="depth_camera">
+                <pose>0 0.0175 0.0125 0 0 0</pose>
+                <update_rate>6</update_rate>
+                <always_on>0</always_on>
+                <camera>
+                    <horizontal_fov>1.51843645</horizontal_fov>
+                    <camera_info_topic>depth_camera_${number}/camera_info</camera_info_topic>
+                    <image>
+                        <width>848</width>
+                        <height>480</height>
+                        <format>R_FLOAT32</format>
+                    </image>
+                    <clip>
+                        <near>0.1</near>
+                        <far>10</far>
+                    </clip>
+                    <lens>
+                        <intrinsics>
+                            <fx>421.61578369140625</fx>
+                            <fy>421.61578369140625</fy>
+                            <cx>422.2854309082031</cx>
+                            <cy>236.57237243652344</cy>
+                            <s>0</s>
+                        </intrinsics>
+                    </lens>
+                </camera>
+                <topic>depth_camera_${number}/image_raw</topic>
+                <gz_frame_id>depth_camera_link_optical</gz_frame_id>
+            </sensor>
+            <!-- <sensor name="semantic_segmentation_camera" type="segmentation">
+                <topic>semantic</topic>
+                <camera>
+                    <segmentation_type>semantic</segmentation_type>
+                    <horizontal_fov>1.57</horizontal_fov>
+                    <image>
+                    <width>800</width>
+                    <height>600</height>
+                    </image>
+                    <clip>
+                    <near>0.1</near>
+                    <far>100</far>
+                    </clip>
+                    <save enabled="true">
+                    <path>segmentation_data/semantic_camera</path>
+                    </save>
+                </camera>
+                <always_on>1</always_on>
+                <update_rate>30</update_rate>
+                <visualize>true</visualize>
+            </sensor> -->
+            <!-- Segmentation camera sensor -->
+            <sensor name="semantic_camera_${number}" type="segmentation">
+                <always_on>1</always_on>
+                <update_rate>10</update_rate>
+                <topic>semantic_camera_${number}</topic>
+                <camera>
+                    <segmentation_type>instance</segmentation_type>
+                    <horizontal_fov>${horizontal_fov}</horizontal_fov>
+                    <camera_info_topic>semantic_camera_${number}/camera_info</camera_info_topic>
+                    <image>
+                    <width>800</width><height>600</height>
+                    </image>
+                    <clip><near>0.1</near><far>100</far></clip>
+                    <save enabled="false"/>
+                </camera>
+                <topic>semantic_camera_${number}/image_raw</topic>
+                <gz_frame_id>semantic_camera_link_optical</gz_frame_id>
+                <visualize>true</visualize>
+            </sensor>
         </gazebo>
     </xacro:macro>
-    <xacro:macro name="camera" params="number x y z r p w width height k1 k2 k3 p1 p2 horizental_fov aspect_ratio">
+    <xacro:macro name="camera" params="number x y z r p w width height k1 k2 k3 p1 p2 horizontal_fov aspect_ratio">
         <xacro:camera_link number="${number}"/>
         <xacro:camera_joint number="${number}" x="${x}" y="${y}" z="${z}" r="${r}" p="${p}" w="${w}"/>
-        <xacro:camera_gazebo number="${number}" width="${width}" height="${height}" k1="${k1}" k2="${k2}" k3="${k3}" p1="${p1}" p2="${p2}" horizental_fov="${horizental_fov}" aspect_ratio="${aspect_ratio}"  />
+        <xacro:camera_gazebo number="${number}" width="${width}" height="${height}" k1="${k1}" k2="${k2}" k3="${k3}" p1="${p1}" p2="${p2}" horizontal_fov="${horizontal_fov}" aspect_ratio="${aspect_ratio}"  />
     </xacro:macro>
 </robot>
