Commit message: - Documentation and presentation: Hamid Ebadi - System integration tests : Pär Aronsson - Overall system diagrams : Anton Stigemyr Hill - Pytorch model for humanoid MoCap : Pär Aronsson - Improved documentation and AutoGluon configuration : Marwa Naili - Demo scenario : Anton Stigemyr Hill

File: simulation/humanoid_robot/model/support/arm_3dof.xacro (robot description, xacro)
@@ -12,5 +12,5 @@
     <!-- twist arm length is the rest of the length to get to 1 meter from end of link 1 -->
     <xacro:property name="twist_arm_length" value="${1-(revolute_arm_length*2)}"/>
-    <link name="arm_base_link">
+    <link name="base_link">
         <visual>
             <geometry>
@@ -99,5 +99,5 @@
     <!-- Fixed joint to slightly raise humanoid before movement -->
     <joint name="base_link1_joint" type="fixed">
-        <parent link="arm_base_link"/>
+        <parent link="base_link"/>
         <child link="link1"/>
         <origin xyz="0 0 ${arm_base_height}" rpy="0 0 0"/>

File: simulation/humanoid_robot/model/support/human_support.xacro (robot description, xacro)
@@ -9,3 +9,11 @@
         <child link="Pelvis"/>
     </joint>
+    <gazebo>
+        <plugin filename="gz-sim-pose-publisher-system" name="gz::sim::systems::PosePublisher">
+            <publish_link_pose>false</publish_link_pose>
+            <publish_collision_pose>false</publish_collision_pose>
+            <publish_visual_pose>false</publish_visual_pose>
+            <publish_nested_model_pose>true</publish_nested_model_pose>
+        </plugin>
+    </gazebo>
 </robot>

File: simulation/humanoid_support_moveit_config/config/human_support.ros2_control.xacro (robot description, xacro)
@@ -1,5 +1,5 @@
 <?xml version="1.0"?>
 <robot xmlns:xacro="http://www.ros.org/wiki/xacro">
-    <xacro:macro name="human_support_ros2_control" params="name initial_positions_file">
+    <xacro:macro name="human_support_ros2_control" params="name initial_positions_file namespace">
         <xacro:property name="initial_positions" value="${load_yaml(initial_positions_file)['initial_positions']}"/>
         <ros2_control name="${name}" type="system">
@@ -343,5 +343,6 @@
           <parameters>$(find humanoid_support_moveit_config)/config/ros2_controllers.yaml</parameters>
           <ros>
-              <namespace>/humanoid</namespace>
+              <!-- <namespace>/humanoid_1</namespace> -->
+              <namespace>/${namespace}</namespace>
               <!-- <remapping>/robot_description:=/humanoid/robot_description</remapping> -->
           </ros>
@@ -354,20 +355,20 @@
         <plugin>gz_ros2_control/GazeboSimSystem</plugin>
     </hardware>
-    <joint name="humanoid_front_left_wheel_joint">
+    <joint name="front_left_wheel_joint">
       <command_interface name="velocity"/>
       <state_interface name="position"/>
       <state_interface name="velocity"/>
     </joint>
-    <joint name="humanoid_rear_left_wheel_joint">
+    <joint name="rear_left_wheel_joint">
       <command_interface name="velocity"/>
       <state_interface name="position"/>
       <state_interface name="velocity"/>
     </joint>
-    <joint name="humanoid_front_right_wheel_joint">
+    <joint name="front_right_wheel_joint">
       <command_interface name="velocity"/>
       <state_interface name="position"/>
       <state_interface name="velocity"/>
     </joint>
-    <joint name="humanoid_rear_right_wheel_joint">
+    <joint name="rear_right_wheel_joint">
       <command_interface name="velocity"/>
       <state_interface name="position"/>

File: simulation/humanoid_support_moveit_config/config/human_support.urdf.xacro (robot description, xacro)
@@ -2,4 +2,5 @@
 <robot xmlns:xacro="http://www.ros.org/wiki/xacro" name="human_support">
     <xacro:arg name="initial_positions_file" default="initial_positions.yaml" />
+    <xacro:arg name="namespace" default="humanoid_1" />
     <!-- Import human_support urdf file -->
     <xacro:include filename="$(find humanoid_robot)/model/support/human_support.xacro" />
@@ -7,4 +8,4 @@
     <xacro:include filename="human_support.ros2_control.xacro" />
     <xacro:include filename="human_support_wheels.urdf.xacro" />
-    <xacro:human_support_ros2_control name="GazeboSimSystem" initial_positions_file="$(arg initial_positions_file)"/>
+    <xacro:human_support_ros2_control name="GazeboSimSystem" initial_positions_file="$(arg initial_positions_file)" namespace="$(arg namespace)"/>
 </robot>

File: simulation/humanoid_support_moveit_config/config/human_support_wheels.urdf.xacro (robot description, xacro)
@@ -30,5 +30,5 @@
     </gazebo>
     <joint name="${wheel_prefix}_wheel_joint" type="continuous">
-      <parent link="humanoid_chassi_link"/>
+      <parent link="chassi_link"/>
       <child link="${wheel_prefix}_wheel_link" />
       <xacro:insert_block name="joint_pose" />
@@ -45,21 +45,21 @@
     </transmission>
   </xacro:macro>
-  <xacro:wheel wheel_prefix="humanoid_front_left">
+  <xacro:wheel wheel_prefix="front_left">
     <origin xyz="${wheelbase/2} ${track/2} ${wheel_vertical_offset}" rpy="0 0 0" />
   </xacro:wheel>
-  <xacro:wheel wheel_prefix="humanoid_front_right">
+  <xacro:wheel wheel_prefix="front_right">
     <origin xyz="${wheelbase/2} ${-track/2} ${wheel_vertical_offset}" rpy="0 0 0" />
   </xacro:wheel>
-  <xacro:wheel wheel_prefix="humanoid_rear_left">
+  <xacro:wheel wheel_prefix="rear_left">
     <origin xyz="${-wheelbase/2} ${track/2} ${wheel_vertical_offset}" rpy="0 0 0" />
   </xacro:wheel>
-  <xacro:wheel wheel_prefix="humanoid_rear_right">
+  <xacro:wheel wheel_prefix="rear_right">
     <origin xyz="${-wheelbase/2} ${-track/2} ${wheel_vertical_offset}" rpy="0 0 0" />
   </xacro:wheel>
-  <joint name="humanoid_base_link_joint" type="fixed">
+  <joint name="base_link_joint" type="fixed">
     <origin xyz="0 0 0" rpy="0 0 0" />
-    <parent link="arm_base_link"/>
-    <child link="humanoid_chassi_link" />
+    <parent link="base_link"/>
+    <child link="chassi_link" />
   </joint>
-  <link name="humanoid_chassi_link"/>
+  <link name="chassi_link"/>
   </robot>

File: simulation/pallet_truck/pallet_truck_description/urdf/pallet_truck.urdf.xacro (robot description, xacro)
@@ -279,3 +279,11 @@
     </gazebo>
   </xacro:if>
+  <gazebo>
+      <plugin filename="gz-sim-pose-publisher-system" name="gz::sim::systems::PosePublisher">
+          <publish_link_pose>false</publish_link_pose>
+          <publish_collision_pose>false</publish_collision_pose>
+          <publish_visual_pose>false</publish_visual_pose>
+          <publish_nested_model_pose>true</publish_nested_model_pose>
+      </plugin>
+  </gazebo>
 </robot>

File: simulation/simlan_gazebo_environment/worlds/ign_simlan_factory.world.xacro (robot description, xacro)
@@ -728,5 +728,5 @@
       <uri>model://eur_pallet</uri>
       <name>pallet_group_dropoff</name>
-      <pose>32.3 6.6 0.001 0 -0 0</pose>
+      <pose>33.0 4.5 0.001 0 -0 0</pose>
     </include>
     <include>

File: simulation/static_agent_launcher/description/agents.urdf.xacro (robot description, xacro)
@@ -8,5 +8,5 @@
         <!-- <xacro:inertial_box mass="0.1" x="0.12" y="0.15" z="0.15"/> -->
     </link>
-    <link name="base_link">
+    <link name="static_agents/base_link">
         <xacro:inertial_box mass="0.1" x="0.12" y="0.15" z="0.15"/>
     </link>
@@ -14,5 +14,5 @@
         <origin xyz="0 0 0" rpy="0 0 0"/>
         <parent link="world"/>
-        <child link="base_link"/>
+        <child link="static_agents/base_link"/>
     </joint>
     <xacro:include filename="camera_config.xacro" />

File: simulation/static_agent_launcher/description/aruco_macros.xacro (robot description, xacro)
@@ -47,5 +47,5 @@
    </xacro:macro>
    <xacro:macro name="aruco" params="number x y z r p w">
-        <xacro:attach_aruco attach_to="base_link" number="${number}" x="${x}" y="${y}" z="${z}" r="${r}" p="${p}" w="${w}"/>
+        <xacro:attach_aruco attach_to="static_agents/base_link" number="${number}" x="${x}" y="${y}" z="${z}" r="${r}" p="${p}" w="${w}"/>
    </xacro:macro>
     <xacro:macro name="attach_aruco" params="attach_to number x y z r p w">

File: simulation/static_agent_launcher/description/camera_config.xacro (robot description, xacro)
@@ -2,12 +2,6 @@
 <!-- =================================== -->
 <robot xmlns:xacro="http://www.ros.org/wiki/xacro">
-<xacro:camera number="162" x="-5.583158189893617" y="1.1215696998181661" z="7.334558192411435" r="1.5153065411297053" p="1.2585498082517528" w="-0.0623840194833805" width="3840" height="2160" k1="-0.3881529379410545" k2="0.21282043348416652" k3="-0.07191487688493671" p1="-0.0003723515252576787" p2="7.348232914337802e-05" horizontal_fov="1.4623791470550955" aspect_ratio="1.7777777777777777" fx="2140.3200768199777" fy="2135.2780770836384" cx="1929.0005479705692" cy="1096.7745783880505"/>
 <xacro:camera number="163" x="6.408863223463873" y="1.0584660310604614" z="7.292500745934432" r="1.26150086062305" p="1.5251520264293401" w="-0.3776042405847099" width="3840" height="2160" k1="-0.38583566587127305" k2="0.2099961443873393" k3="-0.07094931776988343" p1="9.279371221442497e-05" p2="0.00014849011979552266" horizontal_fov="1.4581859532350445" aspect_ratio="1.7777777777777777" fx="2149.369021637226" fy="2145.313127853166" cx="1927.5991222455455" cy="1097.3958400200925"/>
 <xacro:camera number="164" x="19.018611699231805" y="0.5996158690202327" z="7.312413251033552" r="1.5198482458361036" p="1.2025224147143143" w="2.9981981711263943" width="3840" height="2160" k1="-0.3851544658419547" k2="0.2065606446662026" k3="-0.06703301309031716" p1="-8.882469357164693e-05" p2="-0.0002282099854856601" horizontal_fov="1.4620172315943898" aspect_ratio="1.7777777777777777" fx="2141.0994238929516" fy="2137.284406587473" cx="1925.9800217107563" cy="1100.503689897023"/>
 <xacro:camera number="165" x="19.780977546074062" y="-3.5988921587419385" z="7.320450325717854" r="0.21646481266366288" p="1.2312003431796872" w="0.13995159212967984" width="3840" height="2160" k1="-0.3856199901471728" k2="0.20812766168662827" k3="-0.0686518264523881" p1="-0.00023961544692403472" p2="-8.229104930400743e-05" horizontal_fov="1.4615731089914958" aspect_ratio="1.7777777777777777" fx="2142.056225377218" fy="2138.1828027123133" cx="1925.882769040276" cy="1105.8536578341075"/>
-<xacro:camera number="166" x="22.963270174027638" y="4.027979359238905" z="7.419277685692496" r="-1.0558178103115716" p="1.3797771301022628" w="-1.8322918256936183" width="3840" height="2160" k1="-0.38144336503488374" k2="0.19579882600150705" k3="-0.0586530291683016" p1="-0.0002683294214338217" p2="-2.68226954291596e-05" horizontal_fov="1.461834064552691" aspect_ratio="1.7777777777777777" fx="2141.49397483713" fy="2136.455041642565" cx="1929.600290737873" cy="1102.8496242762226"/>
-<xacro:camera number="500" x="2.5" y="-10.0" z="2.0" r="2.220446049250313e-16" p="-4.930380657631324e-32" w="2.220446049250313e-16" width="3840" height="2160" k1="-0.3851544658419547" k2="0.2065606446662026" k3="-0.06703301309031716" p1="-8.882469357164693e-05" p2="-0.0002282099854856601" horizontal_fov="1.4620172315943898" aspect_ratio="1.7777777777777777" fx="2141.0994238929516" fy="2137.284406587473" cx="1925.9800217107563" cy="1100.503689897023"/>
-<xacro:camera number="501" x="5.5" y="-13.0" z="1.9999999999999998" r="0.0" p="-2.220446049250313e-16" w="1.5707963267948966" width="3840" height="2160" k1="-0.3851544658419547" k2="0.2065606446662026" k3="-0.06703301309031716" p1="-8.882469357164693e-05" p2="-0.0002282099854856601" horizontal_fov="1.4620172315943898" aspect_ratio="1.7777777777777777" fx="2141.0994238929516" fy="2137.284406587473" cx="1925.9800217107563" cy="1100.503689897023"/>
-<xacro:camera number="502" x="8.5" y="-10.0" z="2.0" r="-2.220446049250313e-16" p="-4.930380657631324e-32" w="3.141592653589793" width="3840" height="2160" k1="-0.3851544658419547" k2="0.2065606446662026" k3="-0.06703301309031716" p1="-8.882469357164693e-05" p2="-0.0002282099854856601" horizontal_fov="1.4620172315943898" aspect_ratio="1.7777777777777777" fx="2141.0994238929516" fy="2137.284406587473" cx="1925.9800217107563" cy="1100.503689897023"/>
-<xacro:camera number="503" x="5.5" y="-6.999999999999999" z="2.0000000000000004" r="-2.719262146893782e-32" p="2.220446049250313e-16" w="-1.5707963267948968" width="3840" height="2160" k1="-0.3851544658419547" k2="0.2065606446662026" k3="-0.06703301309031716" p1="-8.882469357164693e-05" p2="-0.0002282099854856601" horizontal_fov="1.4620172315943898" aspect_ratio="1.7777777777777777" fx="2141.0994238929516" fy="2137.284406587473" cx="1925.9800217107563" cy="1100.503689897023"/>
 </robot>

File: simulation/static_agent_launcher/description/camera_macros.xacro (robot description, xacro)
@@ -1,5 +1,5 @@
 <robot xmlns:xacro="http://www.ros.org/wiki/xacro">
     <xacro:macro name="camera_link" params="number">
-        <link name="camera_${number}_link">
+        <link name="static_agents/camera_${number}_link">
           <visual>
               <origin xyz="-0.03 0 0" rpy="0 0 0"/>
@@ -20,10 +20,10 @@
         <joint name="camera_${number}_joint" type="fixed">
             <origin xyz="${x} ${y} ${z}" rpy="${r} ${p} ${w}"/>
-            <parent link="base_link"/>
-            <child link="camera_${number}_link"/>
+            <parent link="static_agents/base_link"/>
+            <child link="static_agents/camera_${number}_link"/>
         </joint>
     </xacro:macro>
     <xacro:macro name="camera_gazebo" params="number width height k1 k2 k3 p1 p2 horizontal_fov aspect_ratio fx fy cx cy">
-        <gazebo reference="camera_${number}_link">
+        <gazebo reference="static_agents/camera_${number}_link">
             <!-- Camera Sensor -->
             <sensor name="camera_${number}" type="camera">
