Commit message: fix: namespacing for jackal and pallet_truck

File: simulation/pallet_truck/pallet_truck_description/urdf/pallet_truck.urdf.xacro (robot description, xacro)
@@ -59,5 +59,5 @@
     </gazebo>
     <joint name="${wheel_prefix}_wheel_joint" type="continuous">
-      <parent link="$(arg prefix)_chassis_link"/>
+      <parent link="$(arg prefix)/chassis_link"/>
       <child link="${wheel_prefix}_wheel_link" />
       <xacro:insert_block name="joint_pose" />
@@ -76,23 +76,23 @@
     </transmission>
   </xacro:macro>
-  <xacro:wheel wheel_prefix="$(arg prefix)_front_left">
+  <xacro:wheel wheel_prefix="$(arg prefix)/front_left">
     <origin xyz="${wheelbase/2} ${track/2} ${wheel_vertical_offset}" rpy="0 0 0" />
   </xacro:wheel>
-  <xacro:wheel wheel_prefix="$(arg prefix)_front_right">
+  <xacro:wheel wheel_prefix="$(arg prefix)/front_right">
     <origin xyz="${wheelbase/2} ${-track/2} ${wheel_vertical_offset}" rpy="0 0 0" />
   </xacro:wheel>
-  <xacro:wheel wheel_prefix="$(arg prefix)_rear_left">
+  <xacro:wheel wheel_prefix="$(arg prefix)/rear_left">
     <origin xyz="${-wheelbase/2} ${track/2} ${wheel_vertical_offset}" rpy="0 0 0" />
   </xacro:wheel>
-  <xacro:wheel wheel_prefix="$(arg prefix)_rear_right">
+  <xacro:wheel wheel_prefix="$(arg prefix)/rear_right">
     <origin xyz="${-wheelbase/2} ${-track/2} ${wheel_vertical_offset}" rpy="0 0 0" />
   </xacro:wheel>
   <joint name="scan_joint" type="fixed">
     <origin xyz="0 0 1.5" rpy="0 0 0"/>
-    <parent link="$(arg prefix)_base_link"/>
-    <child link="$(arg prefix)_scan_link"/>
+    <parent link="$(arg prefix)/base_link"/>
+    <child link="$(arg prefix)/scan_link"/>
   </joint>
   <!-- LIDAR -->
-  <link name="$(arg prefix)_scan_link">
+  <link name="$(arg prefix)/scan_link">
       <visual>
       <origin xyz="0 0 0" rpy="0 0 0"/>
@@ -102,11 +102,11 @@
     </visual>
   </link>
-  <link name="$(arg prefix)_base_link"></link>
-  <joint name="$(arg prefix)_base_link_joint" type="fixed">
+  <link name="$(arg prefix)/base_link"></link>
+  <joint name="$(arg prefix)/base_link_joint" type="fixed">
     <origin xyz="0 0 0" rpy="0 0 0" />
-    <parent link="$(arg prefix)_base_link"/>
-    <child link="$(arg prefix)_chassis_link" />
-  </joint>
-  <link name="$(arg prefix)_chassis_link">
+    <parent link="$(arg prefix)/base_link"/>
+    <child link="$(arg prefix)/chassis_link" />
+  </joint>
+  <link name="$(arg prefix)/chassis_link">
   <xacro:if value="${robot_type == 'pallet_truck'}">
     <visual>
@@ -170,5 +170,5 @@
        always points to the "active" IMU. When an upgrade IMU is connected, the
        internal_imu_link should remain, but imu_link should point to the upgrade one. -->
-  <link name="$(arg prefix)_imu_link">
+  <link name="$(arg prefix)/imu_link">
     <inertial>
       <mass value="0.001"/>
@@ -177,11 +177,11 @@
     </inertial>
   </link>
-  <joint name="$(arg prefix)_imu_joint" type="fixed">
-    <parent link="$(arg prefix)_chassis_link" />
-    <child link="$(arg prefix)_imu_link" />
+  <joint name="$(arg prefix)/imu_joint" type="fixed">
+    <parent link="$(arg prefix)/chassis_link" />
+    <child link="$(arg prefix)/imu_link" />
   </joint>
   <!-- TODO Same note as applies to imu_link -->
   <!--
-  <link name="$(arg prefix)_navsat_link">
+  <link name="$(arg prefix)/navsat_link">
     <visual>
       <geometry>
@@ -192,25 +192,25 @@
     </visual>
   </link>
-  <joint name="$(arg prefix)_navsat_joint" type="fixed">
-    <parent link="$(arg prefix)_chassis_link" />
-    <child link="$(arg prefix)_navsat_link" />
+  <joint name="$(arg prefix)/navsat_joint" type="fixed">
+    <parent link="$(arg prefix)/chassis_link" />
+    <child link="$(arg prefix)/navsat_link" />
     <origin xyz="-0.180 0.126 0.1815" />
   </joint>
-  <link name="$(arg prefix)_mid_mount"></link>
-  <joint name="$(arg prefix)_mid_mount_joint" type="fixed">
-    <parent link="$(arg prefix)_chassis_link" />
-    <child link="$(arg prefix)_mid_mount" />
+  <link name="$(arg prefix)/mid_mount"></link>
+  <joint name="$(arg prefix)/mid_mount_joint" type="fixed">
+    <parent link="$(arg prefix)/chassis_link" />
+    <child link="$(arg prefix)/mid_mount" />
     <origin xyz="0 0 ${chassis_height}" />
   </joint>
-  <link name="$(arg prefix)_rear_mount"></link>
-  <joint name="$(arg prefix)_rear_mount_joint" type="fixed">
-    <parent link="$(arg prefix)_mid_mount" />
-    <child link="$(arg prefix)_rear_mount" />
+  <link name="$(arg prefix)/rear_mount"></link>
+  <joint name="$(arg prefix)/rear_mount_joint" type="fixed">
+    <parent link="$(arg prefix)/mid_mount" />
+    <child link="$(arg prefix)/rear_mount" />
     <origin xyz="${-mount_spacing} 0 0" />
   </joint>
-  <link name="$(arg prefix)_front_mount"></link>
-  <joint name="$(arg prefix)_front_mount_joint" type="fixed">
-    <parent link="$(arg prefix)_mid_mount" />
-    <child link="$(arg prefix)_front_mount" />
+  <link name="$(arg prefix)/front_mount"></link>
+  <joint name="$(arg prefix)/front_mount_joint" type="fixed">
+    <parent link="$(arg prefix)/mid_mount" />
+    <child link="$(arg prefix)/front_mount" />
     <origin xyz="${mount_spacing} 0 0" />
   </joint>
@@ -227,20 +227,20 @@
       </xacro:unless>
     </hardware>
-    <joint name="$(arg prefix)_front_left_wheel_joint">
-      <command_interface name="velocity"/>
-      <state_interface name="position"/>
-      <state_interface name="velocity"/>
-    </joint>
-    <joint name="$(arg prefix)_rear_left_wheel_joint">
-      <command_interface name="velocity"/>
-      <state_interface name="position"/>
-      <state_interface name="velocity"/>
-    </joint>
-    <joint name="$(arg prefix)_front_right_wheel_joint">
-      <command_interface name="velocity"/>
-      <state_interface name="position"/>
-      <state_interface name="velocity"/>
-    </joint>
-    <joint name="$(arg prefix)_rear_right_wheel_joint">
+    <joint name="$(arg prefix)/front_left_wheel_joint">
+      <command_interface name="velocity"/>
+      <state_interface name="position"/>
+      <state_interface name="velocity"/>
+    </joint>
+    <joint name="$(arg prefix)/rear_left_wheel_joint">
+      <command_interface name="velocity"/>
+      <state_interface name="position"/>
+      <state_interface name="velocity"/>
+    </joint>
+    <joint name="$(arg prefix)/front_right_wheel_joint">
+      <command_interface name="velocity"/>
+      <state_interface name="position"/>
+      <state_interface name="velocity"/>
+    </joint>
+    <joint name="$(arg prefix)/rear_right_wheel_joint">
       <command_interface name="velocity"/>
       <state_interface name="position"/>

Commit message: release: v3.0.0: jazzy

File: simulation/pallet_truck/pallet_truck_description/urdf/pallet_truck.urdf.xacro (robot description, xacro)
@@ -5,5 +5,5 @@
   <xacro:arg name="namespace" default="pallet_truck" />
   <xacro:property name="robot_type" value="$(arg robot_type)" />
-  <!-- <xacro:property name="prefix" default="$(arg prefix)" /> -->
+  <!-- <xacro:property name="prefix" default="$(arg prefix)"/> -->
   <xacro:arg name="gazebo_controllers" default="$(find pallet_truck_control)/config/control.yaml" />
   <xacro:property name="PI" value="3.1415926535897931" />
@@ -19,4 +19,5 @@
   <xacro:property name="dummy_inertia" value="1e-09"/>
   <xacro:property name="mount_spacing" value="0.120" />
+  <xacro:property name="prefix" value="$(arg prefix)"/>
   <material name="dark_grey"><color rgba="0.2 0.2 0.2 1.0" /></material>
   <material name="light_grey"><color rgba="0.4 0.4 0.4 1.0" /></material>
@@ -88,4 +89,6 @@
     <origin xyz="${-wheelbase/2} ${-track/2} ${wheel_vertical_offset}" rpy="0 0 0" />
   </xacro:wheel>
+ <!-- LIDAR -->
+  <!--
   <joint name="scan_joint" type="fixed">
     <origin xyz="0 0 1.5" rpy="0 0 0"/>
@@ -93,5 +96,4 @@
     <child link="$(arg prefix)/scan_link"/>
   </joint>
-  <!-- LIDAR -->
   <link name="$(arg prefix)/scan_link">
       <visual>
@@ -102,4 +104,5 @@
     </visual>
   </link>
+  -->
   <link name="$(arg prefix)/base_link"></link>
   <joint name="$(arg prefix)/base_link_joint" type="fixed">
@@ -115,7 +118,7 @@
         <mesh filename="file://$(find pallet_truck_description)/meshes/VOLVO_AVG.dae" scale="0.6 0.6 0.6" />
       </geometry>
-        <material name="black" />
-    </visual>
-    <collision>
+      <material name="black" />
+    </visual>
+    <collision name='collision'>
       <origin xyz="0 0 0" rpy="0 0 0"/>
       <geometry>
@@ -147,12 +150,4 @@
       </geometry>
     </collision>
-    <!--
-    <collision>
-      <origin xyz="0 0 ${chassis_height/2}"/>
-      <geometry>
-        <box size="${chassis_length} ${chassis_width} ${chassis_height}"/>
-      </geometry>
-    </collision>
-    -->
     <inertial>
       <!-- Center of mass -->
@@ -248,4 +243,14 @@
     </joint>
   </ros2_control>
+  <xacro:if value="${robot_type == 'pallet_truck'}">
+    <gazebo reference="$(arg prefix)/chassis_link">
+      <sensor name="$(arg prefix)/contact_sensor" type="contact">
+        <always_on>true</always_on>
+        <contact>
+            <collision>${prefix}_base_link_fixed_joint_lump__collision_collision</collision>
+        </contact>
+      </sensor>
+    </gazebo>
+  </xacro:if>
   <!-- Bring in simulation data for Gazebo. -->
   <!-- <xacro:if value="$(arg is_sim)"> -->
@@ -257,3 +262,20 @@
   <!-- Optional custom includes. -->
   <!--<xacro:include filename="$(optenv pallet_truck_URDF_EXTRAS empty.urdf)" />-->
+<!-- This is for the semantic segmentation, to have different labels for pallet truck and forklift-->
+  <xacro:if value="${robot_type == 'forklift'}">
+    <gazebo>
+      <!-- Semantic Segmentation Label Plugin -->
+      <plugin filename="gz-sim-label-system" name="gz::sim::systems::Label">
+        <label>50</label>  <!-- unique ID for forklift -->
+      </plugin>
+    </gazebo>
+  </xacro:if>
+  <xacro:if value="${robot_type == 'pallet_truck'}">
+    <gazebo>
+      <!-- Semantic Segmentation Label Plugin -->
+      <plugin filename="gz-sim-label-system" name="gz::sim::systems::Label">
+        <label>51</label>  <!-- unique ID for pallet truck -->
+      </plugin>
+    </gazebo>
+  </xacro:if>
 </robot>

File: simulation/static_agent_launcher/description/camera_config.xacro (robot description, xacro)
@@ -2,7 +2,8 @@
 <!-- =================================== -->
 <robot xmlns:xacro="http://www.ros.org/wiki/xacro">
-<xacro:camera number="163" x="6.408863223463874" y="1.0584660310604614" z="7.292500745934433" r="1.26150086062305" p="1.5251520264293401" w="-0.3776042405847099" width="3840" height="2160" k1="-0.38583566587127305" k2="0.2099961443873393" k3="-0.07094931776988343" p1="9.279371221442497e-05" p2="0.00014849011979552266" horizontal_fov="1.4581859532350445" aspect_ratio="1.7777777777777777"  />
-<xacro:camera number="164" x="19.018611699231805" y="0.5996158690202326" z="7.312413251033551" r="1.5198482458361036" p="1.2025224147143143" w="2.9981981711263943" width="3840" height="2160" k1="-0.3851544658419547" k2="0.2065606446662026" k3="-0.06703301309031716" p1="-8.882469357164693e-05" p2="-0.0002282099854856601" horizontal_fov="1.4620172315943898" aspect_ratio="1.7777777777777777"  />
-<xacro:camera number="165" x="19.780977546074062" y="-3.598892158741938" z="7.320450325717852" r="0.21646481266366294" p="1.2312003431796872" w="0.13995159212967984" width="3840" height="2160" k1="-0.3856199901471728" k2="0.20812766168662827" k3="-0.0686518264523881" p1="-0.00023961544692403472" p2="-8.229104930400743e-05" horizontal_fov="1.4615731089914958" aspect_ratio="1.7777777777777777"  />
-<xacro:camera number="166" x="22.963270174027635" y="4.027979359238904" z="7.419277685692497" r="-1.0558178103115718" p="1.3797771301022628" w="-1.8322918256936183" width="3840" height="2160" k1="-0.38144336503488374" k2="0.19579882600150705" k3="-0.0586530291683016" p1="-0.0002683294214338217" p2="-2.68226954291596e-05" horizontal_fov="1.461834064552691" aspect_ratio="1.7777777777777777"  />
+<xacro:camera number="162" x="-5.583158189893617" y="1.1215696998181661" z="7.334558192411435" r="1.5153065411297053" p="1.2585498082517528" w="-0.0623840194833805" width="3840" height="2160" k1="-0.3881529379410545" k2="0.21282043348416652" k3="-0.07191487688493671" p1="-0.0003723515252576787" p2="7.348232914337802e-05" horizontal_fov="1.4623791470550955" aspect_ratio="1.7777777777777777" fx="2140.3200768199777" fy="2135.2780770836384" cx="1929.0005479705692" cy="1096.7745783880505"/>
+<xacro:camera number="163" x="6.408863223463873" y="1.0584660310604614" z="7.292500745934432" r="1.26150086062305" p="1.5251520264293401" w="-0.3776042405847099" width="3840" height="2160" k1="-0.38583566587127305" k2="0.2099961443873393" k3="-0.07094931776988343" p1="9.279371221442497e-05" p2="0.00014849011979552266" horizontal_fov="1.4581859532350445" aspect_ratio="1.7777777777777777" fx="2149.369021637226" fy="2145.313127853166" cx="1927.5991222455455" cy="1097.3958400200925"/>
+<xacro:camera number="164" x="19.018611699231805" y="0.5996158690202327" z="7.312413251033552" r="1.5198482458361036" p="1.2025224147143143" w="2.9981981711263943" width="3840" height="2160" k1="-0.3851544658419547" k2="0.2065606446662026" k3="-0.06703301309031716" p1="-8.882469357164693e-05" p2="-0.0002282099854856601" horizontal_fov="1.4620172315943898" aspect_ratio="1.7777777777777777" fx="2141.0994238929516" fy="2137.284406587473" cx="1925.9800217107563" cy="1100.503689897023"/>
+<xacro:camera number="165" x="19.780977546074062" y="-3.5988921587419385" z="7.320450325717854" r="0.21646481266366288" p="1.2312003431796872" w="0.13995159212967984" width="3840" height="2160" k1="-0.3856199901471728" k2="0.20812766168662827" k3="-0.0686518264523881" p1="-0.00023961544692403472" p2="-8.229104930400743e-05" horizontal_fov="1.4615731089914958" aspect_ratio="1.7777777777777777" fx="2142.056225377218" fy="2138.1828027123133" cx="1925.882769040276" cy="1105.8536578341075"/>
+<xacro:camera number="166" x="22.963270174027638" y="4.027979359238905" z="7.419277685692496" r="-1.0558178103115716" p="1.3797771301022628" w="-1.8322918256936183" width="3840" height="2160" k1="-0.38144336503488374" k2="0.19579882600150705" k3="-0.0586530291683016" p1="-0.0002683294214338217" p2="-2.68226954291596e-05" horizontal_fov="1.461834064552691" aspect_ratio="1.7777777777777777" fx="2141.49397483713" fy="2136.455041642565" cx="1929.600290737873" cy="1102.8496242762226"/>
 </robot>

File: simulation/static_agent_launcher/description/camera_macros.xacro (robot description, xacro)
@@ -24,5 +24,5 @@
         </joint>
     </xacro:macro>
-    <xacro:macro name="camera_gazebo" params="number width height k1 k2 k3 p1 p2 horizontal_fov aspect_ratio">
+    <xacro:macro name="camera_gazebo" params="number width height k1 k2 k3 p1 p2 horizontal_fov aspect_ratio fx fy cx cy">
         <gazebo reference="camera_${number}_link">
             <!-- Camera Sensor -->
@@ -35,5 +35,4 @@
                   <horizontal_fov>${horizontal_fov}</horizontal_fov>
                   <camera_info_topic>camera_${number}/camera_info</camera_info_topic>
-                  <aspect_ratio>${aspect_ratio}</aspect_ratio>
                   <image>
                     <width>${width}</width>
@@ -41,8 +40,13 @@
                     <format>R8G8B8</format>
                   </image>
+                <clip>
+                    <near>0.1</near>
+                    <far>100</far>
+                </clip>
                 <lens>
                     <radial_tangential>
                         <k1>${k1}</k1>
                         <k2>${k2}</k2>
+                        <k3>${k3}</k3>
                         <p1>${p1}</p1>
                         <p2>${p2}</p2>
@@ -54,5 +58,4 @@
             </sensor>
             <!-- Depth camera sensor -->
-            <!--
             <sensor name="depth_${number}" type="depth_camera">
                 <pose>0 0.0175 0.0125 0 0 0</pose>
@@ -63,18 +66,18 @@
                     <camera_info_topic>depth_camera_${number}/camera_info</camera_info_topic>
                     <image>
-                        <width>848</width>
-                        <height>480</height>
+                        <width>${width}</width>
+                        <height>${height}</height>
                         <format>R_FLOAT32</format>
                     </image>
                     <clip>
                         <near>0.1</near>
-                        <far>10</far>
+                        <far>100</far>
                     </clip>
                     <lens>
                         <intrinsics>
-                            <fx>421.61578369140625</fx>
-                            <fy>421.61578369140625</fy>
-                            <cx>422.2854309082031</cx>
-                            <cy>236.57237243652344</cy>
+                            <fx>${fx}</fx>
+                            <fy>${fy}</fy>
+                            <cx>${cx}</cx>
+                            <cy>${cy}</cy>
                             <s>0</s>
                         </intrinsics>
@@ -84,28 +87,5 @@
                 <gz_frame_id>depth_camera_link_optical</gz_frame_id>
             </sensor>
-            -->
-            <!-- <sensor name="semantic_segmentation_camera" type="segmentation">
-                <topic>semantic</topic>
-                <camera>
-                    <segmentation_type>semantic</segmentation_type>
-                    <horizontal_fov>1.57</horizontal_fov>
-                    <image>
-                    <width>800</width>
-                    <height>600</height>
-                    </image>
-                    <clip>
-                    <near>0.1</near>
-                    <far>100</far>
-                    </clip>
-                    <save enabled="true">
-                    <path>segmentation_data/semantic_camera</path>
-                    </save>
-                </camera>
-                <always_on>1</always_on>
-                <update_rate>30</update_rate>
-                <visualize>true</visualize>
-            </sensor> -->
             <!-- Segmentation camera sensor -->
-            <!--
             <sensor name="semantic_camera_${number}" type="segmentation">
                 <always_on>1</always_on>
@@ -113,9 +93,9 @@
                 <topic>semantic_camera_${number}</topic>
                 <camera>
-                    <segmentation_type>instance</segmentation_type>
+                    <segmentation_type>semantic</segmentation_type>
                     <horizontal_fov>${horizontal_fov}</horizontal_fov>
                     <camera_info_topic>semantic_camera_${number}/camera_info</camera_info_topic>
                     <image>
-                    <width>800</width><height>600</height>
+                    <width>${width}</width><height>${height}</height>
                     </image>
                     <clip><near>0.1</near><far>100</far></clip>
@@ -126,11 +106,10 @@
                 <visualize>true</visualize>
             </sensor>
-            -->
         </gazebo>
     </xacro:macro>
-    <xacro:macro name="camera" params="number x y z r p w width height k1 k2 k3 p1 p2 horizontal_fov aspect_ratio">
+    <xacro:macro name="camera" params="number x y z r p w width height k1 k2 k3 p1 p2 horizontal_fov aspect_ratio fx fy cx cy">
         <xacro:camera_link number="${number}"/>
         <xacro:camera_joint number="${number}" x="${x}" y="${y}" z="${z}" r="${r}" p="${p}" w="${w}"/>
-        <xacro:camera_gazebo number="${number}" width="${width}" height="${height}" k1="${k1}" k2="${k2}" k3="${k3}" p1="${p1}" p2="${p2}" horizontal_fov="${horizontal_fov}" aspect_ratio="${aspect_ratio}"  />
+        <xacro:camera_gazebo number="${number}" width="${width}" height="${height}" k1="${k1}" k2="${k2}" k3="${k3}" p1="${p1}" p2="${p2}" horizontal_fov="${horizontal_fov}" aspect_ratio="${aspect_ratio}" fx="${fx}" fy="${fy}" cx="${cx}" cy="${cy}" />
     </xacro:macro>
 </robot>
