Commit message: 4.0.1 release: - Working demo video scenario: Hamid Ebadi, Pär Aronsson - Refactor and improve prediction pipeline: Pär Aronsson - Review and update the mocap architecture: Pär Aronsson, Hamid Ebadi - Pipeline for Prediction on real data, images, and videos: Pär Aronsson - Improve motion player: Pär Aronsson - New demo scenario: Pär Aronsson - Unify "single" and "multi" pipeline: Pär Aronsson, Hamid Ebadi - Documentation and presentation (mkdocs, pandas): Hamid Ebadi

File: simulation/pallet_truck/pallet_truck_description/urdf/pallet_truck.urdf.xacro (robot description, xacro)
@@ -144,5 +144,5 @@
         <material name="black" />
     </visual>
-    <collision>
+    <collision name='collision'>
       <origin xyz="-0.5 -0.25 0" rpy="0 0 0"/>
       <geometry>
@@ -243,14 +243,12 @@
     </joint>
   </ros2_control>
-  <xacro:if value="${robot_type == 'pallet_truck'}">
-    <gazebo reference="$(arg prefix)/chassis_link">
-      <sensor name="$(arg prefix)/contact_sensor" type="contact">
-        <always_on>true</always_on>
-        <contact>
-            <collision>${prefix}_base_link_fixed_joint_lump__collision_collision</collision>
-        </contact>
-      </sensor>
-    </gazebo>
-  </xacro:if>
+  <gazebo reference="$(arg prefix)/chassis_link">
+    <sensor name="$(arg prefix)/contact_sensor" type="contact">
+      <always_on>true</always_on>
+      <contact>
+          <collision>${prefix}/base_link_fixed_joint_lump__collision_collision</collision>
+      </contact>
+    </sensor>
+  </gazebo>
   <!-- Bring in simulation data for Gazebo. -->
   <!-- <xacro:if value="$(arg is_sim)"> -->

File: simulation/static_agent_launcher/description/agents.urdf.xacro (robot description, xacro)
@@ -1,4 +1,8 @@
 <?xml version="1.0"?>
 <robot xmlns:xacro="http://www.ros.org/wiki/xacro"  name="robot">
+    <xacro:arg name="camera_update_rate" default="30"/>
+    <xacro:arg name="camera_streams" default="image depth semantic"/>
+    <xacro:property name="camera_streams" value="$(arg camera_streams)" />
+    <xacro:property name="camera_update_rate" value="$(arg camera_update_rate)" />
     <xacro:include filename="properties.xacro" />
     <xacro:include filename="camera_macros.xacro"/>

File: simulation/static_agent_launcher/description/camera_config.xacro (robot description, xacro)
@@ -2,6 +2,8 @@
 <!-- =================================== -->
 <robot xmlns:xacro="http://www.ros.org/wiki/xacro">
-<xacro:camera number="163" x="6.408863223463873" y="1.0584660310604614" z="7.292500745934432" r="1.26150086062305" p="1.5251520264293401" w="-0.3776042405847099" width="3840" height="2160" k1="-0.38583566587127305" k2="0.2099961443873393" k3="-0.07094931776988343" p1="9.279371221442497e-05" p2="0.00014849011979552266" horizontal_fov="1.4581859532350445" aspect_ratio="1.7777777777777777" fx="2149.369021637226" fy="2145.313127853166" cx="1927.5991222455455" cy="1097.3958400200925"/>
 <xacro:camera number="164" x="19.018611699231805" y="0.5996158690202327" z="7.312413251033552" r="1.5198482458361036" p="1.2025224147143143" w="2.9981981711263943" width="3840" height="2160" k1="-0.3851544658419547" k2="0.2065606446662026" k3="-0.06703301309031716" p1="-8.882469357164693e-05" p2="-0.0002282099854856601" horizontal_fov="1.4620172315943898" aspect_ratio="1.7777777777777777" fx="2141.0994238929516" fy="2137.284406587473" cx="1925.9800217107563" cy="1100.503689897023"/>
 <xacro:camera number="165" x="19.780977546074062" y="-3.5988921587419385" z="7.320450325717854" r="0.21646481266366288" p="1.2312003431796872" w="0.13995159212967984" width="3840" height="2160" k1="-0.3856199901471728" k2="0.20812766168662827" k3="-0.0686518264523881" p1="-0.00023961544692403472" p2="-8.229104930400743e-05" horizontal_fov="1.4615731089914958" aspect_ratio="1.7777777777777777" fx="2142.056225377218" fy="2138.1828027123133" cx="1925.882769040276" cy="1105.8536578341075"/>
+<xacro:camera number="166" x="22.963270174027638" y="4.027979359238905" z="7.419277685692496" r="-1.0558178103115716" p="1.3797771301022628" w="-1.8322918256936183" width="3840" height="2160" k1="-0.38144336503488374" k2="0.19579882600150705" k3="-0.0586530291683016" p1="-0.0002683294214338217" p2="-2.68226954291596e-05" horizontal_fov="1.461834064552691" aspect_ratio="1.7777777777777777" fx="2141.49397483713" fy="2136.455041642565" cx="1929.600290737873" cy="1102.8496242762226"/>
+<xacro:camera number="167" x="20.320795688398483" y="8.551222492793519" z="7.698006516690173" r="0.25137394405842073" p="1.2896252866077818" w="-1.4053010395980856" width="3840" height="2160" k1="-0.3838819131967851" k2="0.2010505063378464" k3="-0.062406328638322184" p1="-0.0001384477473404489" p2="-0.0001711681317662323" horizontal_fov="1.45994289873241" aspect_ratio="1.7777777777777777" fx="2145.5723590051794" fy="2141.6133907308695" cx="1928.9381467242947" cy="1102.9142309406184"/>
+<xacro:camera number="168" x="26.791802520963806" y="5.716299217374743" z="3.8958341874803013" r="-0.011612268544003568" p="0.5170306055823943" w="1.5964779037829606" width="3840" height="2160" k1="-0.38226542199738556" k2="0.19688945293158802" k3="-0.05884113267485558" p1="0.00010222372875181348" p2="-0.00019454336997989425" horizontal_fov="1.4570619080710934" aspect_ratio="1.7777777777777777" fx="2151.801940498995" fy="2147.9256682435" cx="1926.074286111512" cy="1097.5030444178685"/>
 </robot>

File: simulation/static_agent_launcher/description/camera_macros.xacro (robot description, xacro)
@@ -1,4 +1,4 @@
 <robot xmlns:xacro="http://www.ros.org/wiki/xacro">
-    <xacro:macro name="camera_link" params="number">
+    <xacro:macro name="camera_link" params="number" >
         <link name="static_agents/camera_${number}_link">
           <visual>
@@ -26,39 +26,45 @@
     <xacro:macro name="camera_gazebo" params="number width height k1 k2 k3 p1 p2 horizontal_fov aspect_ratio fx fy cx cy">
         <gazebo reference="static_agents/camera_${number}_link">
-            <!-- Camera Sensor -->
+            <xacro:define_cameras camera_streams="${camera_streams}" camera_update_rate="${camera_update_rate}" number="${number}" width="${width}" height="${height}" k1="${k1}" k2="${k2}" k3="${k3}" p1="${p1}" p2="${p2}" horizontal_fov="${horizontal_fov}" aspect_ratio="${aspect_ratio}" fx="${fx}" fy="${fy}" cx="${cx}" cy="${cy}" />
+        </gazebo>
+    </xacro:macro>
+    <xacro:macro name="define_cameras" params="camera_streams camera_update_rate number width height k1 k2 k3 p1 p2 horizontal_fov aspect_ratio fx fy cx cy">
+        <!-- Image camera -->
+        <xacro:if value="${camera_streams.find('image') != -1}">
             <sensor name="camera_${number}" type="camera">
                 <always_on>true</always_on>
                 <visualize>true</visualize>
-                <update_rate>20</update_rate>
+                <update_rate>${camera_update_rate}</update_rate>
                 <camera name="intel_realsense_r200">
-                  <!-- <segmentation_type>instance</segmentation_type> -->
-                  <horizontal_fov>${horizontal_fov}</horizontal_fov>
-                  <camera_info_topic>camera_${number}/camera_info</camera_info_topic>
-                  <image>
-                    <width>${width}</width>
-                    <height>${height}</height>
-                    <format>R8G8B8</format>
-                  </image>
-                <clip>
-                    <near>0.1</near>
-                    <far>100</far>
-                </clip>
-                <lens>
-                    <radial_tangential>
-                        <k1>${k1}</k1>
-                        <k2>${k2}</k2>
-                        <k3>${k3}</k3>
-                        <p1>${p1}</p1>
-                        <p2>${p2}</p2>
-                    </radial_tangential>
-                </lens>
+                    <horizontal_fov>${horizontal_fov}</horizontal_fov>
+                    <camera_info_topic>camera_${number}/camera_info</camera_info_topic>
+                    <image>
+                        <width>${width}</width>
+                        <height>${height}</height>
+                        <format>R8G8B8</format>
+                    </image>
+                    <clip>
+                        <near>0.1</near>
+                        <far>100</far>
+                    </clip>
+                    <lens>
+                        <radial_tangential>
+                            <k1>${k1}</k1>
+                            <k2>${k2}</k2>
+                            <k3>${k3}</k3>
+                            <p1>${p1}</p1>
+                            <p2>${p2}</p2>
+                        </radial_tangential>
+                    </lens>
                 </camera>
                 <topic>camera_${number}/image_raw</topic>
                 <gz_frame_id>camera_link_optical</gz_frame_id>
             </sensor>
-            <!-- Depth camera sensor -->
+        </xacro:if>
+        <!-- Depth camera -->
+        <xacro:if value="${camera_streams.find('depth') != -1}">
             <sensor name="depth_${number}" type="depth_camera">
                 <pose>0 0.0175 0.0125 0 0 0</pose>
-                <update_rate>6</update_rate>
+                <update_rate>${camera_update_rate}</update_rate>
                 <always_on>0</always_on>
                 <camera>
@@ -87,8 +93,10 @@
                 <gz_frame_id>depth_camera_link_optical</gz_frame_id>
             </sensor>
-            <!-- Segmentation camera sensor -->
+        </xacro:if>
+        <!-- Semantic camera -->
+        <xacro:if value="${camera_streams.find('semantic') != -1}">
             <sensor name="semantic_camera_${number}" type="segmentation">
                 <always_on>1</always_on>
-                <update_rate>10</update_rate>
+                <update_rate>${camera_update_rate}</update_rate>
                 <topic>semantic_camera_${number}</topic>
                 <camera>
@@ -106,5 +114,5 @@
                 <visualize>true</visualize>
             </sensor>
-        </gazebo>
+        </xacro:if>
     </xacro:macro>
     <xacro:macro name="camera" params="number x y z r p w width height k1 k2 k3 p1 p2 horizontal_fov aspect_ratio fx fy cx cy">

File: simulation/static_agent_launcher/description/properties.xacro (robot description, xacro)
@@ -21,4 +21,3 @@
     <xacro:property name="camera_resolution_width" value="1920"/>
     <xacro:property name="camera_resolution_height" value="1080"/>
-    <xacro:property name="camera_update_rate" value="30"/>
 </robot>
