Commit message: feat: multiple bots (pallete truck or forklift) in different namespaces

File: simulation/pallet_truck/pallet_truck_description/urdf/aruco.xacro (robot description, xacro)
@@ -2,6 +2,7 @@
 <robot name="infobot_infobot"
     xmlns:xacro="http://ros.org/wiki/xacro">
+    <xacro:property name="aruco_id" value="0" />
     <xacro:macro name="aruco_link" params="number">
-        <link name="aruco_${number}_link">
+        <link name="$(arg prefix)_aruco_${number}_link">
             <visual>
                 <origin xyz="0 0 0" rpy="0 0 ${PI}"/>
@@ -13,8 +14,8 @@
         <joint name="aruco_${number}_joint" type="fixed">
             <origin xyz="-0.8 0 1.30" rpy="0 0 0"/>
-            <parent link="pallet_truck_base_link"/>
-            <child link="aruco_${number}_link"/>
+            <parent link="$(arg prefix)_base_link"/>
+            <child link="$(arg prefix)_aruco_${number}_link"/>
         </joint>
-        <gazebo reference="aruco_${number}_link">
+        <gazebo reference="$(arg prefix)_aruco_${number}_link">
             <static>true</static>
             <visual name="aruco_front_face">
@@ -27,6 +28,6 @@
                     <pbr>
                         <metal>
-                            <albedo_map>model://aruco/materials/textures/12.png</albedo_map>
-                            <name>aruco_0</name>
+                            <albedo_map>model://aruco/materials/textures/${number}.png</albedo_map>
+                            <name>"aruco_${number}"</name>
                         </metal>
                     </pbr>
@@ -35,4 +36,4 @@
         </gazebo>
     </xacro:macro>
-    <xacro:aruco_link number="12" />
+    <xacro:aruco_link number="$(arg aruco_id)" />
 </robot>

File: simulation/pallet_truck/pallet_truck_description/urdf/pallet_truck.urdf.xacro (robot description, xacro)
@@ -3,4 +3,6 @@
   <xacro:arg name="is_sim" default="true" />
   <xacro:arg name="prefix" default="pallet_truck" />
+  <xacro:arg name="namespace" default="pallet_truck" />
+  <xacro:property name="robot_type" value="$(arg robot_type)" />
   <!-- <xacro:property name="prefix" default="$(arg prefix)" /> -->
   <xacro:arg name="gazebo_controllers" default="$(find pallet_truck_control)/config/control.yaml" />
@@ -107,4 +109,5 @@
   </joint>
   <link name="$(arg prefix)_chassis_link">
+  <xacro:if value="${robot_type == 'pallet_truck'}">
     <visual>
       <origin xyz="0 0 0" rpy="0 0 0"/>
@@ -118,4 +121,28 @@
       <geometry>
         <mesh filename="file://$(find pallet_truck_description)/meshes/VOLVO_AVG.dae" scale="0.6 0.6 0.6" />
+      </geometry>
+    </collision>
+    <inertial>
+      <!-- Center of mass -->
+      <origin xyz="0.012  0.002 0.067" rpy="0 0 0"/>
+      <mass value="16.523"/>
+      <inertia
+        ixx="0.3136" ixy="-0.0008" ixz="0.0164"
+        iyy="0.3922" iyz="-0.0009"
+        izz="0.4485"/>
+    </inertial>
+  </xacro:if>
+  <xacro:if value="${robot_type == 'forklift'}">
+    <visual>
+      <origin xyz="-0.5 -0.25 0" rpy="0 0 0"/>
+      <geometry>
+        <mesh filename="file://$(find simlan_gazebo_environment)/models/forklift_robot/forklift_robot_description/meshes/base_link.dae" scale="0.6 0.6 0.6" />
+      </geometry>
+        <material name="black" />
+    </visual>
+    <collision>
+      <origin xyz="-0.5 -0.25 0" rpy="0 0 0"/>
+      <geometry>
+        <mesh filename="file://$(find simlan_gazebo_environment)/models/forklift_robot/forklift_robot_description/meshes/base_link.dae" scale="0.6 0.6 0.6" />
       </geometry>
     </collision>
@@ -137,4 +164,5 @@
         izz="0.4485"/>
     </inertial>
+  </xacro:if>
   </link>
   <!-- TODO Make this internal_imu_link or something, and use a mixed-in xacro

File: simulation/static_agent_launcher/description/agents.urdf.xacro (robot description, xacro)
@@ -17,5 +17,5 @@
     </joint>
     <xacro:include filename="camera_config.xacro" />
-    <xacro:aruco number="1" x="7" y="3" z="0.001" r="0" p="0" w="0"/>
-    <xacro:aruco number="2" x="6" y="0" z="0.001" r="0" p="0" w="0"/>
+   <!-- <xacro:aruco number="20" x="7" y="3" z="0.001" r="0" p="0" w="0"/> -->
+   <!-- <xacro:aruco number="30" x="6" y="0" z="0.001" r="0" p="0" w="0"/> -->
 </robot>

File: simulation/static_agent_launcher/description/camera_macros.xacro (robot description, xacro)
@@ -54,4 +54,5 @@
             </sensor>
             <!-- Depth camera sensor -->
+            <!--
             <sensor name="depth_${number}" type="depth_camera">
                 <pose>0 0.0175 0.0125 0 0 0</pose>
@@ -83,4 +84,5 @@
                 <gz_frame_id>depth_camera_link_optical</gz_frame_id>
             </sensor>
+            -->
             <!-- <sensor name="semantic_segmentation_camera" type="segmentation">
                 <topic>semantic</topic>
@@ -105,4 +107,5 @@
             </sensor> -->
             <!-- Segmentation camera sensor -->
+            <!--
             <sensor name="semantic_camera_${number}" type="segmentation">
                 <always_on>1</always_on>
@@ -123,4 +126,5 @@
                 <visualize>true</visualize>
             </sensor>
+            -->
         </gazebo>
     </xacro:macro>

Commit message: fix errors in tf trees and namespace missmatches. Simulation is running

File: simulation/pallet_truck/pallet_truck_description/urdf/aruco.xacro (robot description, xacro)
@@ -4,5 +4,5 @@
     <xacro:property name="aruco_id" value="0" />
     <xacro:macro name="aruco_link" params="number">
-        <link name="$(arg prefix)_aruco_${number}_link">
+        <link name="$(arg prefix)/aruco_${number}_link">
             <visual>
                 <origin xyz="0 0 0" rpy="0 0 ${PI}"/>
@@ -14,8 +14,8 @@
         <joint name="aruco_${number}_joint" type="fixed">
             <origin xyz="-0.8 0 1.30" rpy="0 0 0"/>
-            <parent link="$(arg prefix)_base_link"/>
-            <child link="$(arg prefix)_aruco_${number}_link"/>
+            <parent link="$(arg prefix)/base_link"/>
+            <child link="$(arg prefix)/aruco_${number}_link"/>
         </joint>
-        <gazebo reference="$(arg prefix)_aruco_${number}_link">
+        <gazebo reference="$(arg prefix)/aruco_${number}_link">
             <static>true</static>
             <visual name="aruco_front_face">

Commit message: v5.1.0 : merge gitlab to github

File: simulation/pallet_truck/pallet_truck_description/urdf/aruco.xacro (robot description, xacro)
@@ -4,5 +4,5 @@
     <xacro:property name="aruco_id" value="0" />
     <xacro:macro name="aruco_link" params="number">
-        <link name="$(arg prefix)/aruco_${number}_link">
+        <link name="aruco_${number}_link">
             <visual>
                 <origin xyz="0 0 0" rpy="0 0 ${PI}"/>
@@ -14,8 +14,8 @@
         <joint name="aruco_${number}_joint" type="fixed">
             <origin xyz="-0.8 0 1.30" rpy="0 0 0"/>
-            <parent link="$(arg prefix)/base_link"/>
-            <child link="$(arg prefix)/aruco_${number}_link"/>
+            <parent link="base_link"/>
+            <child link="aruco_${number}_link"/>
         </joint>
-        <gazebo reference="$(arg prefix)/aruco_${number}_link">
+        <gazebo reference="aruco_${number}_link">
             <static>true</static>
             <visual name="aruco_front_face">

File: simulation/pallet_truck/pallet_truck_description/urdf/pallet_truck.urdf.xacro (robot description, xacro)
@@ -1,9 +1,8 @@
 <?xml version="1.0"?>
-<robot name="pallet_truck" xmlns:xacro="http://www.ros.org/wiki/xacro">
+<robot name="pallet_truck"
+  xmlns:xacro="http://www.ros.org/wiki/xacro">
   <xacro:arg name="is_sim" default="true" />
-  <xacro:arg name="prefix" default="pallet_truck" />
   <xacro:arg name="namespace" default="pallet_truck" />
   <xacro:property name="robot_type" value="$(arg robot_type)" />
-  <!-- <xacro:property name="prefix" default="$(arg prefix)"/> -->
   <xacro:arg name="gazebo_controllers" default="$(find pallet_truck_control)/config/control.yaml" />
   <xacro:property name="PI" value="3.1415926535897931" />
@@ -19,9 +18,17 @@
   <xacro:property name="dummy_inertia" value="1e-09"/>
   <xacro:property name="mount_spacing" value="0.120" />
-  <xacro:property name="prefix" value="$(arg prefix)"/>
-  <material name="dark_grey"><color rgba="0.2 0.2 0.2 1.0" /></material>
-  <material name="light_grey"><color rgba="0.4 0.4 0.4 1.0" /></material>
-  <material name="yellow"><color rgba="0.8 0.8 0.0 1.0" /></material>
-  <material name="black"><color rgba="0.15 0.15 0.15 1.0" /></material>
+  <xacro:property name="namespace" value="$(arg namespace)"/>
+  <material name="dark_grey">
+    <color rgba="0.2 0.2 0.2 1.0" />
+  </material>
+  <material name="light_grey">
+    <color rgba="0.4 0.4 0.4 1.0" />
+  </material>
+  <material name="yellow">
+    <color rgba="0.8 0.8 0.0 1.0" />
+  </material>
+  <material name="black">
+    <color rgba="0.15 0.15 0.15 1.0" />
+  </material>
   <xacro:include filename="$(find pallet_truck_description)/urdf/aruco.xacro"/>
   <xacro:include filename="$(find pallet_truck_description)/urdf/pallet_truck.gazebo" />
@@ -44,8 +51,5 @@
         <origin xyz="0 0 0" rpy="0 0 0"/>
         <mass value="0.477"/>
-        <inertia
-          ixx="0.0013" ixy="0" ixz="0"
-          iyy="0.0024" iyz="0"
-          izz="0.0013"/>
+        <inertia ixx="0.0013" ixy="0" ixz="0" iyy="0.0024" iyz="0" izz="0.0013"/>
       </inertial>
     </link>
@@ -60,5 +64,5 @@
     </gazebo>
     <joint name="${wheel_prefix}_wheel_joint" type="continuous">
-      <parent link="$(arg prefix)/chassis_link"/>
+      <parent link="chassis_link"/>
       <child link="${wheel_prefix}_wheel_link" />
       <xacro:insert_block name="joint_pose" />
@@ -77,17 +81,17 @@
     </transmission>
   </xacro:macro>
-  <xacro:wheel wheel_prefix="$(arg prefix)/front_left">
+  <xacro:wheel wheel_prefix="front_left">
     <origin xyz="${wheelbase/2} ${track/2} ${wheel_vertical_offset}" rpy="0 0 0" />
   </xacro:wheel>
-  <xacro:wheel wheel_prefix="$(arg prefix)/front_right">
+  <xacro:wheel wheel_prefix="front_right">
     <origin xyz="${wheelbase/2} ${-track/2} ${wheel_vertical_offset}" rpy="0 0 0" />
   </xacro:wheel>
-  <xacro:wheel wheel_prefix="$(arg prefix)/rear_left">
+  <xacro:wheel wheel_prefix="rear_left">
     <origin xyz="${-wheelbase/2} ${track/2} ${wheel_vertical_offset}" rpy="0 0 0" />
   </xacro:wheel>
-  <xacro:wheel wheel_prefix="$(arg prefix)/rear_right">
+  <xacro:wheel wheel_prefix="rear_right">
     <origin xyz="${-wheelbase/2} ${-track/2} ${wheel_vertical_offset}" rpy="0 0 0" />
   </xacro:wheel>
- <!-- LIDAR -->
+  <!-- LIDAR -->
   <!--
   <joint name="scan_joint" type="fixed">
@@ -105,59 +109,53 @@
   </link>
   -->
-  <link name="$(arg prefix)/base_link"></link>
-  <joint name="$(arg prefix)/base_link_joint" type="fixed">
+  <link name="base_link"></link>
+  <joint name="base_link_joint" type="fixed">
     <origin xyz="0 0 0" rpy="0 0 0" />
-    <parent link="$(arg prefix)/base_link"/>
-    <child link="$(arg prefix)/chassis_link" />
-  </joint>
-  <link name="$(arg prefix)/chassis_link">
-  <xacro:if value="${robot_type == 'pallet_truck'}">
-    <visual>
-      <origin xyz="0 0 0" rpy="0 0 0"/>
-      <geometry>
-        <mesh filename="file://$(find pallet_truck_description)/meshes/VOLVO_AVG.dae" scale="0.6 0.6 0.6" />
-      </geometry>
-      <material name="black" />
-    </visual>
-    <collision name='collision'>
-      <origin xyz="0 0 0" rpy="0 0 0"/>
-      <geometry>
-        <mesh filename="file://$(find pallet_truck_description)/meshes/VOLVO_AVG.dae" scale="0.6 0.6 0.6" />
-      </geometry>
-    </collision>
-    <inertial>
-      <!-- Center of mass -->
-      <origin xyz="0.012  0.002 0.067" rpy="0 0 0"/>
-      <mass value="16.523"/>
-      <inertia
-        ixx="0.3136" ixy="-0.0008" ixz="0.0164"
-        iyy="0.3922" iyz="-0.0009"
-        izz="0.4485"/>
-    </inertial>
-  </xacro:if>
-  <xacro:if value="${robot_type == 'forklift'}">
-    <visual>
-      <origin xyz="-0.5 -0.25 0" rpy="0 0 0"/>
-      <geometry>
-        <mesh filename="file://$(find simlan_gazebo_environment)/models/forklift_robot/forklift_robot_description/meshes/base_link.dae" scale="0.6 0.6 0.6" />
-      </geometry>
+    <parent link="base_link"/>
+    <child link="chassis_link" />
+  </joint>
+  <link name="chassis_link">
+    <xacro:if value="${robot_type == 'pallet_truck'}">
+      <visual>
+        <origin xyz="0 0 0" rpy="0 0 0"/>
+        <geometry>
+          <mesh filename="file://$(find pallet_truck_description)/meshes/VOLVO_AVG.dae" scale="0.6 0.6 0.6" />
+        </geometry>
         <material name="black" />
-    </visual>
-    <collision name='collision'>
-      <origin xyz="-0.5 -0.25 0" rpy="0 0 0"/>
-      <geometry>
-        <mesh filename="file://$(find simlan_gazebo_environment)/models/forklift_robot/forklift_robot_description/meshes/base_link.dae" scale="0.6 0.6 0.6" />
-      </geometry>
-    </collision>
-    <inertial>
-      <!-- Center of mass -->
-      <origin xyz="0.012  0.002 0.067" rpy="0 0 0"/>
-      <mass value="16.523"/>
-      <inertia
-        ixx="0.3136" ixy="-0.0008" ixz="0.0164"
-        iyy="0.3922" iyz="-0.0009"
-        izz="0.4485"/>
-    </inertial>
-  </xacro:if>
+      </visual>
+      <collision name='collision'>
+        <origin xyz="0 0 0" rpy="0 0 0"/>
+        <geometry>
+          <mesh filename="file://$(find pallet_truck_description)/meshes/VOLVO_AVG.dae" scale="0.6 0.6 0.6" />
+        </geometry>
+      </collision>
+      <inertial>
+        <!-- Center of mass -->
+        <origin xyz="0.012  0.002 0.067" rpy="0 0 0"/>
+        <mass value="16.523"/>
+        <inertia ixx="0.3136" ixy="-0.0008" ixz="0.0164" iyy="0.3922" iyz="-0.0009" izz="0.4485"/>
+      </inertial>
+    </xacro:if>
+    <xacro:if value="${robot_type == 'forklift'}">
+      <visual>
+        <origin xyz="-0.5 -0.25 0" rpy="0 0 0"/>
+        <geometry>
+          <mesh filename="file://$(find simlan_gazebo_environment)/models/forklift_robot/forklift_robot_description/meshes/base_link.dae" scale="0.6 0.6 0.6" />
+        </geometry>
+        <material name="black" />
+      </visual>
+      <collision name='collision'>
+        <origin xyz="-0.5 -0.25 0" rpy="0 0 0"/>
+        <geometry>
+          <mesh filename="file://$(find simlan_gazebo_environment)/models/forklift_robot/forklift_robot_description/meshes/base_link.dae" scale="0.6 0.6 0.6" />
+        </geometry>
+      </collision>
+      <inertial>
+        <!-- Center of mass -->
+        <origin xyz="0.012  0.002 0.067" rpy="0 0 0"/>
+        <mass value="16.523"/>
+        <inertia ixx="0.3136" ixy="-0.0008" ixz="0.0164" iyy="0.3922" iyz="-0.0009" izz="0.4485"/>
+      </inertial>
+    </xacro:if>
   </link>
   <!-- TODO Make this internal_imu_link or something, and use a mixed-in xacro
@@ -165,5 +163,5 @@
        always points to the "active" IMU. When an upgrade IMU is connected, the
        internal_imu_link should remain, but imu_link should point to the upgrade one. -->
-  <link name="$(arg prefix)/imu_link">
+  <link name="imu_link">
     <inertial>
       <mass value="0.001"/>
@@ -172,7 +170,7 @@
     </inertial>
   </link>
-  <joint name="$(arg prefix)/imu_joint" type="fixed">
-    <parent link="$(arg prefix)/chassis_link" />
-    <child link="$(arg prefix)/imu_link" />
+  <joint name="imu_joint" type="fixed">
+    <parent link="chassis_link" />
+    <child link="imu_link" />
   </joint>
   <!-- TODO Same note as applies to imu_link -->
@@ -222,20 +220,20 @@
       </xacro:unless>
     </hardware>
-    <joint name="$(arg prefix)/front_left_wheel_joint">
-      <command_interface name="velocity"/>
-      <state_interface name="position"/>
-      <state_interface name="velocity"/>
-    </joint>
-    <joint name="$(arg prefix)/rear_left_wheel_joint">
-      <command_interface name="velocity"/>
-      <state_interface name="position"/>
-      <state_interface name="velocity"/>
-    </joint>
-    <joint name="$(arg prefix)/front_right_wheel_joint">
-      <command_interface name="velocity"/>
-      <state_interface name="position"/>
-      <state_interface name="velocity"/>
-    </joint>
-    <joint name="$(arg prefix)/rear_right_wheel_joint">
+    <joint name="front_left_wheel_joint">
+      <command_interface name="velocity"/>
+      <state_interface name="position"/>
+      <state_interface name="velocity"/>
+    </joint>
+    <joint name="rear_left_wheel_joint">
+      <command_interface name="velocity"/>
+      <state_interface name="position"/>
+      <state_interface name="velocity"/>
+    </joint>
+    <joint name="front_right_wheel_joint">
+      <command_interface name="velocity"/>
+      <state_interface name="position"/>
+      <state_interface name="velocity"/>
+    </joint>
+    <joint name="rear_right_wheel_joint">
       <command_interface name="velocity"/>
       <state_interface name="position"/>
@@ -243,9 +241,9 @@
     </joint>
   </ros2_control>
-  <gazebo reference="$(arg prefix)/chassis_link">
-    <sensor name="$(arg prefix)/contact_sensor" type="contact">
+  <gazebo reference="chassis_link">
+    <sensor name="contact_sensor" type="contact">
       <always_on>true</always_on>
       <contact>
-          <collision>${prefix}/base_link_fixed_joint_lump__collision_collision</collision>
+        <collision>${namespace}/base_link_fixed_joint_lump__collision_collision</collision>
       </contact>
     </sensor>
@@ -260,10 +258,10 @@
   <!-- Optional custom includes. -->
   <!--<xacro:include filename="$(optenv pallet_truck_URDF_EXTRAS empty.urdf)" />-->
-<!-- This is for the semantic segmentation, to have different labels for pallet truck and forklift-->
+  <!-- This is for the semantic segmentation, to have different labels for pallet truck and forklift-->
   <xacro:if value="${robot_type == 'forklift'}">
     <gazebo>
       <!-- Semantic Segmentation Label Plugin -->
       <plugin filename="gz-sim-label-system" name="gz::sim::systems::Label">
-        <label>50</label>  <!-- unique ID for forklift -->
+        <label>50</label>        <!-- unique ID for forklift -->
       </plugin>
     </gazebo>
@@ -273,15 +271,15 @@
       <!-- Semantic Segmentation Label Plugin -->
       <plugin filename="gz-sim-label-system" name="gz::sim::systems::Label">
-        <label>51</label>  <!-- unique ID for pallet truck -->
+        <label>51</label>        <!-- unique ID for pallet truck -->
       </plugin>
     </gazebo>
   </xacro:if>
   <gazebo>
-      <plugin filename="gz-sim-pose-publisher-system" name="gz::sim::systems::PosePublisher">
-          <publish_link_pose>false</publish_link_pose>
-          <publish_collision_pose>false</publish_collision_pose>
-          <publish_visual_pose>false</publish_visual_pose>
-          <publish_nested_model_pose>true</publish_nested_model_pose>
-      </plugin>
+    <plugin filename="gz-sim-pose-publisher-system" name="gz::sim::systems::PosePublisher">
+      <publish_link_pose>false</publish_link_pose>
+      <publish_collision_pose>false</publish_collision_pose>
+      <publish_visual_pose>false</publish_visual_pose>
+      <publish_nested_model_pose>true</publish_nested_model_pose>
+    </plugin>
   </gazebo>
 </robot>
