Commit message: chore: Improve documentation and refactoring code

File: simulation/simlan_gazebo_environment/worlds/ign_simlan_factory.world.xacro (robot description, xacro)
@@ -1,4 +1,5 @@
 <?xml version='1.0' encoding='ASCII'?>
-<sdf version="1.8">
+<sdf version="1.8" xmlns:xacro="http://www.ros.org/wiki/xacro">
+  <xacro:property name="world_setup" value="$(arg world_setup)" />
     <world name="default">
     <gravity>0 0 -9.8</gravity>
@@ -123,19 +124,20 @@
       <pose>8.80 -14.4 0.0005 0 0 0</pose>
     </include>
-    <include>
-      <uri>model://volvo_AVG</uri>
-      <pose>-4 -4 0 0 0 0</pose>
-    </include>
 <!-- ******************** Factory ******************** -->
-    <include>
+    <xacro:if value="${world_setup=='light' or world_setup=='medium' or world_setup=='default'}">
+      <include>
         <uri>model://factory</uri>
         <pose>1.3 -1.4 0 0 0 0</pose>
-    </include>
+      </include>
+    </xacro:if>
 <!-- ******************** Truck ******************** -->
-    <include>
+    <xacro:if value="${world_setup=='medium' or world_setup=='default'}">
+      <include>
         <uri>model://truck</uri>
         <pose>18.0 16.0 0 0 0 0</pose>
-    </include>
+      </include>
+    </xacro:if>
 <!-- ******************** Hazard Lines ******************** -->
+    <xacro:if value="${world_setup=='light' or world_setup=='medium' or world_setup=='default'}">
     <include>
       <static>1</static>
@@ -198,5 +200,7 @@
       <pose>39.69 8.51 0.001 0 0 1.57075</pose>
     </include>
+    </xacro:if>
 <!-- ******************** Railing ******************** -->
+    <xacro:if value="${world_setup=='medium' or world_setup=='default'}">
     <include>
       <static>1</static>
@@ -768,5 +772,7 @@
       <pose>36.3 24.6 1.45 0 0 0</pose>
     </include>
+  </xacro:if>
 <!-- ******************** Objects for data collection ******************** -->
+  <xacro:if value="${world_setup=='default'}">
     <include>
       <uri>model://box_1185x785x1010</uri>
@@ -1597,5 +1603,5 @@
     </include>
 <!-- NEWBOX -->
+</xacro:if>
   </world>
-  <plugin name="gazebo_ros_api_plugin" filename="libgazebo_ros_api_plugin.so"/>
 </sdf>

Commit message: v5.1.4 : ur10, refactore
- add simulation real time factor to config
- UR10 & Robotiq gripper
- refactor control.sh
- refactor build scripts
- add dynorobotics documentation

File: simulation/simlan_gazebo_environment/worlds/ign_simlan_factory.world.xacro (robot description, xacro)
@@ -1,41 +1,31 @@
 <?xml version='1.0' encoding='ASCII'?>
-<sdf version="1.8" xmlns:xacro="http://www.ros.org/wiki/xacro">
+<sdf version="1.8"
+  xmlns:xacro="http://www.ros.org/wiki/xacro">
   <xacro:property name="world_setup" value="$(arg world_setup)" />
-    <world name="default">
+  <xacro:property name="real_time_factor" value="$(arg real_time_factor)" />
+  <world name="default">
     <gravity>0 0 -9.8</gravity>
     <physics type='ode'>
-  <max_step_size>0.01</max_step_size>           <!-- 10 ms per step -->
-  <real_time_update_rate>100</real_time_update_rate> <!-- 100 steps/sec -->
-  <real_time_factor>1</real_time_factor>        <!-- real-time sim -->
-  <max_contacts>10</max_contacts>
-</physics>
-    <plugin
-        filename="gz-sim-physics-system"
-        name="gz::sim::systems::Physics">
+      <max_step_size>0.01</max_step_size>      <!-- 10 ms per step -->
+      <real_time_update_rate>100</real_time_update_rate>      <!-- 100 steps/sec -->
+      <real_time_factor>${real_time_factor}</real_time_factor>      <!-- real-time sim -->
+      <max_contacts>10</max_contacts>
+    </physics>
+    <plugin filename="gz-sim-physics-system" name="gz::sim::systems::Physics">
     </plugin>
-    <plugin
-        filename="gz-sim-user-commands-system"
-        name="gz::sim::systems::UserCommands">
+    <plugin filename="gz-sim-user-commands-system" name="gz::sim::systems::UserCommands">
     </plugin>
-    <plugin
-        filename="gz-sim-scene-broadcaster-system"
-        name="gz::sim::systems::SceneBroadcaster">
+    <plugin filename="gz-sim-scene-broadcaster-system" name="gz::sim::systems::SceneBroadcaster">
     </plugin>
-    <plugin
-        filename="gz-sim-sensors-system"
-        name="gz::sim::systems::Sensors">
-    <render_engine>ogre2</render_engine>
+    <plugin filename="gz-sim-sensors-system" name="gz::sim::systems::Sensors">
+      <render_engine>ogre2</render_engine>
     </plugin>
-    <plugin
-        filename="gz-sim-imu-system"
-        name="gz::sim::systems::Imu">
+    <plugin filename="gz-sim-imu-system" name="gz::sim::systems::Imu">
     </plugin>
-    <plugin filename="gz-sim-contact-system"
-        name="gz::sim::systems::Contact">
+    <plugin filename="gz-sim-contact-system" name="gz::sim::systems::Contact">
     </plugin>
-    <plugin filename="gz-sim-triggered-publisher-system"
-        name="gz::sim::systems::TriggeredPublisher">
+    <plugin filename="gz-sim-triggered-publisher-system" name="gz::sim::systems::TriggeredPublisher">
     </plugin>
-<!-- ******************** Scene & Sun ******************** -->
+    <!-- ******************** Scene & Sun ******************** -->
     <scene>
       <ambient>1 1 1 1</ambient>
@@ -44,5 +34,5 @@
       <grid>false</grid>
     </scene>
-<!--
+    <!--
     <light name='amber_light' type='point'>
       <pose>0 0 1 0 0 0</pose>
@@ -97,40 +87,40 @@
 -->
     <light type="directional" name="sun">
-        <cast_shadows>false</cast_shadows>
-        <pose>0 0.1 10 0 0 0</pose>
-        <diffuse>0.8 0.8 0.8 1</diffuse>
-        <specular>0.2 0.2 0.2 1</specular>
-        <attenuation>
-            <range>1000</range>
-            <constant>0.9</constant>
-            <linear>0.01</linear>
-            <quadratic>0.001</quadratic>
-        </attenuation>
-        <direction>0.1 0.1 -0.9</direction>
+      <cast_shadows>false</cast_shadows>
+      <pose>0 0.1 10 0 0 0</pose>
+      <diffuse>0.8 0.8 0.8 1</diffuse>
+      <specular>0.2 0.2 0.2 1</specular>
+      <attenuation>
+        <range>1000</range>
+        <constant>0.9</constant>
+        <linear>0.01</linear>
+        <quadratic>0.001</quadratic>
+      </attenuation>
+      <direction>0.1 0.1 -0.9</direction>
     </light>
-<!-- ******************** Ground ******************** -->
+    <!-- ******************** Ground ******************** -->
     <xacro:if value="${world_setup=='empty'}">
-    <include>
+      <include>
         <uri>model://ground_plane</uri>
         <pose>10 -10.0 0 0 0 0</pose>
-    </include>
+      </include>
     </xacro:if>
     <xacro:if value="${world_setup=='light' or world_setup=='medium' or world_setup=='default'}">
-    <include>
+      <include>
         <uri>model://ground_collision</uri>
         <pose>1.3 -1.4 0 0 0 0</pose>
-    </include>
-    <include>
+      </include>
+      <include>
         <uri>model://ground_visual_updated</uri>
         <pose>1.3 -1.4 0 0 0 0</pose>
-    </include>
-    <include>
-      <static>1</static>
-      <uri>model://concrete_ground</uri>
-      <name>concrete_ground</name>
-      <pose>8.80 -14.4 0.0005 0 0 0</pose>
-    </include>
+      </include>
+      <include>
+        <static>1</static>
+        <uri>model://concrete_ground</uri>
+        <name>concrete_ground</name>
+        <pose>8.80 -14.4 0.0005 0 0 0</pose>
+      </include>
     </xacro:if>
-<!-- ******************** Factory ******************** -->
+    <!-- ******************** Factory ******************** -->
     <xacro:if value="${world_setup=='light' or world_setup=='medium' or world_setup=='default'}">
       <include>
@@ -139,5 +129,5 @@
       </include>
     </xacro:if>
-<!-- ******************** Truck ******************** -->
+    <!-- ******************** Truck ******************** -->
     <xacro:if value="${world_setup=='medium' or world_setup=='default'}">
       <include>
@@ -146,271 +136,343 @@
       </include>
     </xacro:if>
-<!-- ******************** Hazard Lines ******************** -->
+    <!-- ******************** Hazard Lines ******************** -->
     <xacro:if value="${world_setup=='light' or world_setup=='medium' or world_setup=='default'}">
-    <include>
-      <static>1</static>
-      <uri>model://hazard_lines_striped</uri>
-      <name>hazard_line_1</name>
-      <pose>-26.4 0.1 0.001 0 0 0</pose>
-    </include>
-    <include>
-      <static>1</static>
-      <uri>model://hazard_lines_striped</uri>
-      <name>hazard_line_2_rotated</name>
-      <pose>-7.5 -0.16 0.001 0 0 0.73</pose>
-    </include>
-    <include>
-      <static>1</static>
-      <uri>model://hazard_lines_striped</uri>
-      <name>hazard_line_3_rotated</name>
-      <pose>11.2 0.1 0.001 0 0 -0.2</pose>
-    </include>
-    <include>
-      <static>1</static>
-      <uri>model://hazard_lines</uri>
-      <name>hazard_line_4</name>
-      <pose>16.2 -2 0.001 0 0 1.57075</pose>
-    </include>
-    <include>
-      <static>1</static>
-      <uri>model://hazard_lines</uri>
-      <name>hazard_line_5</name>
-      <pose>23 -2 0.001 0 0 1.57075</pose>
-    </include>
-    <include>
-      <static>1</static>
-      <uri>model://hazard_lines</uri>
-      <name>hazard_line_6</name>
-      <pose>14.68 9.81 0.001 0 0 1.57075</pose>
-    </include>
-    <include>
-      <static>1</static>
-      <uri>model://hazard_lines</uri>
-      <name>hazard_line_7</name>
-      <pose>21.47 9.14 0.001 0 0 1.38</pose>
-    </include>
-    <include>
-      <static>1</static>
-      <uri>model://hazard_lines_striped_scaled</uri>
-      <name>hazard_line_8_rotated_scaled</name>
-      <pose>27.07 8.51 0.001 0 0 1.57075</pose>
-    </include>
-    <include>
-      <static>1</static>
-      <uri>model://hazard_lines</uri>
-      <name>hazard_line_9</name>
-      <pose>32.91 8.51 0.001 0 0 1.57075</pose>
-    </include>
-    <include>
-      <static>1</static>
-      <uri>model://hazard_lines</uri>
-      <name>hazard_line_10</name>
-      <pose>39.69 8.51 0.001 0 0 1.57075</pose>
-    </include>
+      <include>
+        <static>1</static>
+        <uri>model://hazard_lines_striped</uri>
+        <name>hazard_line_1</name>
+        <pose>-26.4 0.1 0.001 0 0 0</pose>
+      </include>
+      <include>
+        <static>1</static>
+        <uri>model://hazard_lines_striped</uri>
+        <name>hazard_line_2_rotated</name>
+        <pose>-7.5 -0.16 0.001 0 0 0.73</pose>
+      </include>
+      <include>
+        <static>1</static>
+        <uri>model://hazard_lines_striped</uri>
+        <name>hazard_line_3_rotated</name>
+        <pose>11.2 0.1 0.001 0 0 -0.2</pose>
+      </include>
+      <include>
+        <static>1</static>
+        <uri>model://hazard_lines</uri>
+        <name>hazard_line_4</name>
+        <pose>16.2 -2 0.001 0 0 1.57075</pose>
+      </include>
+      <include>
+        <static>1</static>
+        <uri>model://hazard_lines</uri>
+        <name>hazard_line_5</name>
+        <pose>23 -2 0.001 0 0 1.57075</pose>
+      </include>
+      <include>
+        <static>1</static>
+        <uri>model://hazard_lines</uri>
+        <name>hazard_line_6</name>
+        <pose>14.68 9.81 0.001 0 0 1.57075</pose>
+      </include>
+      <include>
+        <static>1</static>
+        <uri>model://hazard_lines</uri>
+        <name>hazard_line_7</name>
+        <pose>21.47 9.14 0.001 0 0 1.38</pose>
+      </include>
+      <include>
+        <static>1</static>
+        <uri>model://hazard_lines_striped_scaled</uri>
+        <name>hazard_line_8_rotated_scaled</name>
+        <pose>27.07 8.51 0.001 0 0 1.57075</pose>
+      </include>
+      <include>
+        <static>1</static>
+        <uri>model://hazard_lines</uri>
+        <name>hazard_line_9</name>
+        <pose>32.91 8.51 0.001 0 0 1.57075</pose>
+      </include>
+      <include>
+        <static>1</static>
+        <uri>model://hazard_lines</uri>
+        <name>hazard_line_10</name>
+        <pose>39.69 8.51 0.001 0 0 1.57075</pose>
+      </include>
     </xacro:if>
-<!-- ******************** Railing ******************** -->
+    <!-- ******************** Railing ******************** -->
     <xacro:if value="${world_setup=='medium' or world_setup=='default'}">
-    <include>
-      <static>1</static>
-      <uri>model://railing</uri>
-      <name>railing_1</name>
-      <pose>19.93 2.53 0.001 0 0 0</pose>
-    </include>
-    <include>
-      <static>1</static>
-      <uri>model://railing</uri>
-      <name>railing_2</name>
-      <pose>22.39 -2.95 0.001 0 0 1.57075</pose>
-    </include>
-    <include>
-      <static>1</static>
-      <uri>model://railing</uri>
-      <name>railing_3</name>
-      <pose>22.39 -5.46 0.001 0 0 1.57075</pose>
-    </include>
-    <include>
-      <static>1</static>
-      <uri>model://railing</uri>
-      <name>railing_4</name>
-      <pose>26.33 4.95 0.001 0 0 -2.356125</pose>
-    </include>
-    <include>
-      <static>1</static>
-      <uri>model://railing</uri>
-      <name>railing_5</name>
-      <pose>26.33 4.95 0.15 0 0 -2.356125</pose>
-    </include>
-    <include>
-      <static>1</static>
-      <uri>model://railing</uri>
-      <name>railing_6</name>
-      <pose>26.33 4.95 0.3 0 0 -2.356125</pose>
-    </include>
-    <include>
-      <static>1</static>
-      <uri>model://railing</uri>
-      <name>railing_7</name>
-      <pose>27.3 5.35 0.001 0 0 -3.1415</pose>
-    </include>
-    <include>
-      <static>1</static>
-      <uri>model://railing</uri>
-      <name>railing_8</name>
-      <pose>28.5 5.35 0.001 0 0 -3.1415</pose>
-    </include>
-    <include>
-      <static>1</static>
-      <uri>model://railing</uri>
-      <name>railing_9</name>
-      <pose>29.7 5.35 0.001 0 0 -3.1415</pose>
-    </include>
-    <include>
-      <static>1</static>
-      <uri>model://railing</uri>
-      <name>railing_10</name>
-      <pose>30.9 5.35 0.001 0 0 -3.1415</pose>
-    </include>
-    <include>
-      <static>1</static>
-      <uri>model://railing</uri>
-      <name>railing_11</name>
-      <pose>32.1 5.35 0.001 0 0 -3.1415</pose>
-    </include>
-    <include>
-      <static>1</static>
-      <uri>model://railing</uri>
-      <name>railing_12</name>
-      <pose>32.73 4.72 0.001 0 0 1.57075</pose>
-    </include>
-    <include>
-      <static>1</static>
-      <uri>model://railing</uri>
-      <name>railing_13</name>
-      <pose>19.93 7.07 0.001 0 0 3.1415</pose>
-    </include>
-<!-- ******************** objects ******************** -->
-    <include>
-      <static>1</static>
-      <uri>model://electrical_box</uri>
-      <name>electrical_box</name>
-      <pose>28.89 4 0.001 0 0 3.1415</pose>
-    </include>
-    <include>
-      <static>1</static>
-      <uri>model://blue_cabinet</uri>
-      <name>blue_cabinet</name>
-      <pose>26.95 4.26 0.001 0 0 -1.96</pose>
-    </include>
-    <include>
-      <static>1</static>
-      <uri>model://table</uri>
-      <name>table</name>
-      <pose>40.3 0.35 0.001 0 0 0</pose>
-    </include>
-<!-- ******************** Shelves 0 ******************** -->
-    <include>
-      <static>1</static>
-      <uri>model://shelf</uri>
-      <name>shelf_wall_0_17</name>
-      <pose>19.3 -5.9 0.001 0 0 0</pose>
-    </include>
-<!-- ******************** Shelves 1 ******************** -->
-    <include>
-      <static>1</static>
-      <uri>model://shelf</uri>
-      <name>shelf_wall_1_2</name>
-      <pose>-25.7 -3.4 0.001 0 0 0</pose>
-    </include>
-    <include>
-      <static>1</static>
-      <uri>model://shelf</uri>
-      <name>shelf_wall_1_3</name>
-      <pose>-22.7 -3.4 0.001 0 0 0</pose>
-    </include>
-    <include>
-      <static>1</static>
-      <uri>model://shelf</uri>
-      <name>shelf_wall_1_4</name>
-      <pose>-19.7 -3.4 0.001 0 0 0</pose>
-    </include>
-    <include>
-      <static>1</static>
-      <uri>model://shelf</uri>
-      <name>shelf_wall_1_5</name>
-      <pose>-16.7 -3.4 0.001 0 0 0</pose>
-    </include>
-    <include>
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